File: SmallAvionic/Joyce/Joyce.kicad_sch (KiCad schematic)
At the start: 0 parts

Commit message: not finished smallavionic Joyce
Parts:
- added U1: STM32F103C8Tx, Package_QFP:LQFP-48_7x7mm_P0.5mm, symbol MCU_ST_STM32F1:STM32F103C8Tx
- added U2: BMP390, symbol symbolbmp390test:bmp390
- added U3: BMI088, Package_LGA:Bosch_LGA-16_4.5x3mm_P0.5mm_LayoutBorder7x1y_ClockwisePinNumbering, symbol Sensor_Motion:BMI088
- added U4: W25Q128JVS, Package_SO:SOIC-8_5.3x5.3mm_P1.27mm, symbol Memory_Flash:W25Q128JVS
Connections:
- new net: U1.22 (PB11), U4.1 (~{CS})
- new net: U1.27 (PB14), U4.2 (DO/IO_{1})
- new net: U1.26 (PB13), U4.5 (DI/IO_{0})
- new net: U1.25 (PB12), U4.6 (CLK)
- new net: U1.14 (PA4), U2.6 (CSB), U3.14 (~{CSB1})
- new net: U1.15 (PA5), U2.2 (SCK), U3.8 (SCK/SCL)
- new net: U1.16 (PA6), U2.5 (SDO), U3.15 (SDO1)
- new net: U1.17 (PA7), U2.4 (SDI), U3.9 (SDI/SDA)
- new net: U1.23 (VSS), U1.35 (VSS), U1.47 (VSS)
- new net: U3.2 (GNDA), U3.4 (GNDA)
