File: SmallAvionic/Joyce/Joyce.kicad_sch (KiCad schematic)
At the start: 0 parts

Commit message: Joyce push 1/19
Parts:
- added U1: STM32F103C8Tx, Package_QFP:LQFP-48_7x7mm_P0.5mm, symbol MCU_ST_STM32F1:STM32F103C8Tx
Connections:
- new net: U1.23 (VSS), U1.35 (VSS), U1.47 (VSS)
Changed lines of the file:
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@@
 	(generator "eeschema")
 	(generator_version "9.0")
-	(paper "A4")
+	(paper "A2")
+	(symbol
+		(lib_id "MCU_ST_STM32F1:STM32F103C8Tx")
+		(at 73.66 66.04 0)
+		(unit 1)
+		(exclude_from_sim no)
+		(in_bom yes)
+		(on_board yes)
+		(dnp no)
+		(fields_autoplaced yes)
+		(property "Reference" "U1"
+			(at 78.3433 106.68 0)
+			(effects
+				(font
+					(size 1.27 1.27)
+				)
+				(justify left)
+			)
+		)
+		(property "Value" "STM32F103C8Tx"
+			(at 78.3433 109.22 0)
+			(effects
+				(font
+					(size 1.27 1.27)
+				)
+				(justify left)
+			)
+		)
+		(property "Footprint" "Package_QFP:LQFP-48_7x7mm_P0.5mm"
+			(at 58.42 104.14 0)
+			(effects
+				(font
+					(size 1.27 1.27)
+				)
+				(justify right)
+				(hide yes)
+			)
+		)
+		(property "Datasheet" "https://www.st.com/resource/en/datasheet/stm32f103c8.pdf"
+			(at 73.66 66.04 0)
+			(effects
+				(font
+					(size 1.27 1.27)
+				)
+				(hide yes)
+			)
+		)
+		(property "Description" "STMicroelectronics Arm Cortex-M3 MCU, 64KB flash, 20KB RAM, 72 MHz, 2.0-3.6V, 37 GPIO, LQFP48"
+			(at 73.66 66.04 0)
+			(effects
+				(font
+					(size 1.27 1.27)
+				)
+				(hide yes)
+			)
+		)
+		(pin "46"
+		)
+		(pin "25"
+		)
+		(pin "23"
+		)
+		(pin "44"
+		)
+		(pin "41"
+		)
+		(pin "45"
+		)
+		(pin "3"
+		)
+		(pin "26"
+		)
+		(pin "28"
+		)
+		(pin "5"
+		)
+		(pin "6"
+		)
+		(pin "18"
+		)
+		(pin "2"
+		)
+		(pin "4"
+		)
+		(pin "42"
+		)
+		(pin "43"
+		)
+		(pin "1"
+		)
+		(pin "27"
+		)
+		(pin "24"
+		)
+		(pin "20"
+		)
+		(pin "19"
+		)
+		(pin "7"
+		)
+		(pin "39"
+		)
+		(pin "40"
+		)
+		(pin "21"
+		)
+		(pin "22"
+		)
+		(pin "36"
+		)
+		(pin "12"
+		)
+		(pin "38"
+		)
+		(pin "9"
+		)
+		(pin "34"
+		)
+		(pin "13"
+		)
+		(pin "47"
+		)
+		(pin "8"
+		)
+		(pin "10"
+		)
+		(pin "14"
+		)
+		(pin "29"
+		)
+		(pin "16"
+		)
+		(pin "31"
+		)
+		(pin "11"
+		)
+		(pin "48"
+		)
+		(pin "15"
+		)
+		(pin "17"
+		)
+		(pin "30"
+		)
+		(pin "32"
+		)
+		(pin "35"
+		)
+		(pin "33"
+		)
+		(pin "37"
+		)
+		(instances
+			(project ""
+				(path "/f50f988d-d5d1-4e7d-a554-31b4af09afe7"
+					(reference "U1")
+					(unit 1)
+				)
+			)
+		)
+	)
 	(sheet_instances
 		(path "/"
