File: SmallAvionic/Joyce/Joyce.kicad_sch (KiCad schematic)
At the start: 6 parts, among them IC1 BMP390, U1 STM32F103C8Tx

Commit message: Joyce push 1/26
Parts:
- added C1, C2: 100nF, symbol Device:C
- added C3: 1.0uF, SparkFun_Magnetometer_MMC5983MA_Qwiic_Micro:0402-TIGHT, symbol SparkFun_Magnetometer_MMC5983MA_Qwiic_Micro-eagle-import:1.0UF-0402T-16V-10%
- added C4: 104, symbol Device:C
- added C5: 10uF, SparkFun_Magnetometer_MMC5983MA_Qwiic_Micro:0402-TIGHT, symbol SparkFun_Magnetometer_MMC5983MA_Qwiic_Micro-eagle-import:10UF-0402T-6.3V-20%
- added D1: RED, SparkFun_Magnetometer_MMC5983MA_Qwiic_Micro:LED-0402, symbol SparkFun_Magnetometer_MMC5983MA_Qwiic_Micro-eagle-import:LED-RED_0402
- added D3: LED, symbol Device:LED
- added I2C_PU0: S_MODE, SparkFun_Magnetometer_MMC5983MA_Qwiic_Micro:SMT-JUMPER_3_2-NC_TRACE_SILK, symbol SparkFun_Magnetometer_MMC5983MA_Qwiic_Micro-eagle-import:JUMPER-SMT_3_2-NC_TRAC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
- added J1: QWIIC_RIGHT_ANGLE, SparkFun_Magnetometer_MMC5983MA_Qwiic_Micro:JST04_1MM_RA, symbol SparkFun_Magnetometer_MMC5983MA_Qwiic_Micro-eagle-import:QWIIC_CONNECTORJS-1MM
- added J2, J4: CONN_01_1MM, SparkFun_Magnetometer_MMC5983MA_Qwiic_Micro:1X01_1MM_NO_SILK, symbol SparkFun_Magnetometer_MMC5983MA_Qwiic_Micro-eagle-import:CONN_01_1MM
- added JP1, JP2, JP3: SolderJumper_2_Bridged, symbol Jumper:SolderJumper_2_Bridged
- added LED0: JUMPER-SMT_2_NC_TRACE_SILK, SparkFun_Magnetometer_MMC5983MA_Qwiic_Micro:SMT-JUMPER_2_NC_TRACE_SILK, symbol SparkFun_Magnetometer_MMC5983MA_Qwiic_Micro-eagle-import:JUMPER-SMT_2_NC_TRACE_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
- added R2, R3: 2.2k, SparkFun_Magnetometer_MMC5983MA_Qwiic_Micro:0402-TIGHT, symbol SparkFun_Magnetometer_MMC5983MA_Qwiic_Micro-eagle-import:2.2KOHM-0402T-1/16W-1%
- added R2: 1k, SparkFun_Magnetometer_MMC5983MA_Qwiic_Micro:0402-TIGHT, symbol SparkFun_Magnetometer_MMC5983MA_Qwiic_Micro-eagle-import:1KOHM-0402T-1/16W-1%
- added R5: 1k, symbol Device:R
- added R7: 100k, SparkFun_Magnetometer_MMC5983MA_Qwiic_Micro:0402-TIGHT, symbol SparkFun_Magnetometer_MMC5983MA_Qwiic_Micro-eagle-import:100KOHM-0402T-1/16W-1%
- added TP1, TP2, TP3, TP5: TEST-POINT3, SparkFun_Magnetometer_MMC5983MA_Qwiic_Micro:PAD.03X.03, symbol SparkFun_Magnetometer_MMC5983MA_Qwiic_Micro-eagle-import:TEST-POINT3
- added U2: ~, symbol New_Library:BMi088
- added U3: ~, symbol New_Library:_1
- added U4: MMC5983MA_QFN16, SparkFun_Magnetometer_MMC5983MA_Qwiic_Micro:LGA-16-3X3MM-4X4PINS, symbol SparkFun_Magnetometer_MMC5983MA_Qwiic_Micro-eagle-import:MMC5983MA_QFN16
- added U5: W25Q128JVE, Package_SON:WSON-8-1EP_8x6mm_P1.27mm_EP3.4x4.3mm, symbol Memory_Flash:W25Q128JVE
Connections:
- net 3.3V: now also C3.1, I2C_PU0.2, J1.2, R2.2, R7.2, TP1.1, U4.13 (VDDIO), U4.2 (VDD)
- net CS: now also U2.14 (CSB1), U5.1 (~{CS})
- net GND: now also C3.2, C5.2, J1.1, J4.1, LED0.1, TP5.1, U4.11 (GND), U4.9 (GND)
- net INT: now also J2.1, U4.15 (INT)
- new net: C5.1, U4.10 (CAP)
- new net: U4.12 (NC), U4.14 (NC), U4.3 (NC), U4.6 (NC), U4.7 (NC), U4.8 (NC)
- new net: R7.1, U4.4 (~{SPI_CS})
- new net: I2C_PU0.3, R2.2
- new net: C2.1, JP2.1 (A), U2.3 (VDD)
- new net: I2C_PU0.1, R3.2
- new net: C1.1, JP1.1 (A), U2.11 (VDDIO)
- new net: D1.C, LED0.2
- new net: D1.A, R2.1
- new net: D3.2 (A), R5.1
- new net CLK: U5.6 (CLK)
- new net DI: U5.5 (DI/IO_{0})
- new net DO: U5.2 (DO/IO_{1})
- new net GNDREF: C1.2, C2.2, C4.2, D3.1 (K), U2.4 (GNDA), U2.6 (GNDIO), U3.3 (GND), U5.4 (GND)
- new net GPIO2/INT1: U2.16 (INT1)
- new net GPIO3/INT2: U2.12 (INT3)
- new net GPIO4: U2.5 (CSB2)
- new net GPIO5: U2.7 (PS)
- new net INT A: JP3.1 (A)
- new net INT2_A: U2.1 (INT2)
- new net INT4 G: JP3.2 (B), U2.13 (INT4)
- new net PROM RW: U3.1 (IO)
- new net SCK/SCL: U2.8 (SCx)
- new net SCL: J1.4, R3.1, TP3.1, U4.1 (SCL/SCK)
- new net SDA: J1.3, R2.1, TP2.1, U4.16 (SDA/SDI)
- new net SDI/SDA: U2.9 (SDx)
- new net SDO: U2.10 (SDO2), U2.15 (SDO1)
- new net VCC: C4.1, R5.2, U5.3 (~{WP}/IO_{2}), U5.7 (~{HOLD}/~{RESET}/IO_{3}), U5.8 (VCC)
- new net VDD: JP2.2 (B)
Other:
- note added: "BMI088"
- note added: "Connectors"
- note added: "Cut trace to disconnect Power LED."
- note added: "Cut traces to remove I2C pull-up resistors."
- note added: "I2C address: 0x30"
- note added: "Jumpers"
- note added: "Magnetometer - MMC5983MA"
- note added: "PTH connectors only accept 22AWG or smaller"
- note added: "Testpoints"
- note added: "VDD Range: 2.8V - 3.6V VDDIO Range: 2.8V - 3.6V"
