File: SmallAvionic/Ray/Ray.kicad_sch (KiCad schematic)
At the start: 0 parts

Commit message: Ray push 1/19
Parts:
- added C1, C3, C4: C, symbol Device:C
- added D1, D2, D3: 1N4007, Diode_THT:D_DO-41_SOD81_P10.16mm_Horizontal, symbol Diode:1N4007
- added R1, R2, R3, R4: R, symbol Device:R
- added U1: STM32F103C8Tx, Package_QFP:LQFP-48_7x7mm_P0.5mm, symbol MCU_ST_STM32F1:STM32F103C8Tx
- added U2: BMI088, Package_LGA:Bosch_LGA-16_4.5x3mm_P0.5mm_LayoutBorder7x1y_ClockwisePinNumbering, symbol Sensor_Motion:BMI088
Connections:
- new net: U1.23 (VSS), U1.35 (VSS), U1.47 (VSS)
- new net +3V3: C1.1, C3.1, U2.11 (VDDIO), U2.14 (~{CSB1}), U2.3 (VDD), U2.7 (PS)
- new net AD_0: U2.10 (SDO2)
- new net AD_1: U2.15 (SDO1)
- new net GND: C1.2, C3.2, U2.2 (GNDA), U2.4 (GNDA), U2.6 (GNDIO)
- new net SCL_3v3: U2.8 (SCK/SCL)
- new net SDA_3v3: U2.9 (SDI/SDA)
- no-connect marks 0 -> 1
