File: SmallAvionic/Ray/Ray.kicad_sch (KiCad schematic)
At the start: 52 parts, among them Q1 NMOS, Q2 NMOS, Q3 BSS138, Q4 BSS138, U1 STM32F103C8Tx, U2 BMI088, U3 AP2112K-3.3, U4 XC6206PxxxMR, U5 W25Q128JVS, U6 W25Q128JVE, U7 TPS62142

Commit message: 1/23 complement
Connections:
- net FSW is gone; now on an unnamed net: C15.1, L1.2, R21.1, U7.14 (VOS)
- net 3v3: now also U7.8 (DEF)
Other:
- moved on the sheet: C, C8, C9
