File: SmallAvionic/Ray/Ray.kicad_sch (KiCad schematic)
At the start: 133 parts, among them J1 Boot_mode_pin, J2 USB_C_Receptacle_USB2.0_16P, J3 Conn_01x04, J5 Conn_01x02, Q1 NMOS, Q2 NMOS, Q3 BSS138, Q4 BSS138, Q5 TSM3481CX6 RFG, Q6 TSM3481CX6 RFG, SW1 SW_Push, U1 LD1117S33TR_SOT223, U1 STM32F103C8Tx, U10 TPS54538RQFR, U11 BMI088, U12 STM32F103C8Tx, U13 BMI088, U2 BMI088, U3 AP2112K-3.3, U4 XC6206PxxxMR, U5 W25Q128JVS, U6 W25Q128JVE, U7 TPS62142, U8 STM32F405VGTx, U9 LTC4412xS6, Y1 8Mhz

Commit message: 4/20grounglast
Parts:
- removed 10uF: C, symbol Device:C
- removed 1uF: ~, symbol Device:C
- removed 2.7K (x2): R, symbol Device:R
- removed C, C8: 10uF, symbol Device:C
- removed C16: 10u, symbol Device:C
- removed C17, C18, C19, C21, C23: 100n, symbol Device:C
- removed C22, C24: 4.7u, symbol Device:C
- removed C33, C34: 100nF, symbol Device:C
- removed D2: 1N4148, Diode_THT:D_DO-35_SOD27_P7.62mm_Horizontal, symbol Diode:1N4148
- removed D3: LED, symbol Device:LED
- removed D4: TVS, symbol Device:D_TVS_Filled
- removed D5: G_5V, symbol Device:LED
- removed D6: B_3V3, symbol Device:LED
- removed I2C_PU0: S_MODE, SparkFun_Magnetometer_MMC5983MA_Qwiic_Micro:SMT-JUMPER_3_2-NC_TRACE_SILK, symbol SparkFun_Magnetometer_MMC5983MA_Qwiic_Micro-eagle-import:JUMPER-SMT_3_2-NC_TRAC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
- removed L2: 6.8u, symbol Device:L
- removed LED0: JUMPER-SMT_2_NC_TRACE_SILK, SparkFun_Magnetometer_MMC5983MA_Qwiic_Micro:SMT-JUMPER_2_NC_TRACE_SILK, symbol SparkFun_Magnetometer_MMC5983MA_Qwiic_Micro-eagle-import:JUMPER-SMT_2_NC_TRACE_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
- removed Q1, Q2: NMOS, symbol Simulation_SPICE:NMOS
- removed Q3, Q4: BSS138, Package_TO_SOT_SMD:SOT-23, symbol Transistor_FET:BSS138
- removed Q5, Q6: TSM3481CX6 RFG, Package_TO_SOT_SMD:SOT-23, symbol Transistor_FET:IRLML6402
- removed R10, R11, R9: 10K, symbol Device:R
- removed R12: 100K, symbol Device:R
- removed R30, R34: 100k, symbol Device:R
- removed R31: 220k, symbol Device:R
- removed R32: 1M, symbol Device:R
- removed R33: 30k, symbol Device:R
- removed R36, R37: 22ohm, symbol Device:R
- removed U1: LD1117S33TR_SOT223, Package_TO_SOT_SMD:SOT-223-3_TabPin2, symbol Regulator_Linear:LD1117S33TR_SOT223
- removed U10: TPS54538RQFR, VQFN-HR9_RQF_TEX, symbol Small_av_tony_lib:TPS54538RQFR
- removed U11, U13, U2: BMI088, Package_LGA:Bosch_LGA-16_4.5x3mm_P0.5mm_LayoutBorder7x1y_ClockwisePinNumbering, symbol Sensor_Motion:BMI088
- removed U12: STM32F103C8Tx, Package_QFP:LQFP-48_7x7mm_P0.5mm, symbol MCU_ST_STM32F1:STM32F103C8Tx
- removed U3: AP2112K-3.3, Package_TO_SOT_SMD:SOT-23-5, symbol Regulator_Linear:AP2112K-3.3
- removed U4: XC6206PxxxMR, Package_TO_SOT_SMD:SOT-23-3, symbol Regulator_Linear:XC6206PxxxMR
- removed U5: W25Q128JVS, Package_SO:SOIC-8_5.3x5.3mm_P1.27mm, symbol Memory_Flash:W25Q128JVS
- removed U6: W25Q128JVE, Package_SON:WSON-8-1EP_8x6mm_P1.27mm_EP3.4x4.3mm, symbol Memory_Flash:W25Q128JVE
- removed U7: TPS62142, Package_DFN_QFN:VQFN-16-1EP_3x3mm_P0.5mm_EP1.68x1.68mm_ThermalVias, symbol Regulator_Switching:TPS62142
- removed U8: STM32F405VGTx, Package_QFP:LQFP-100_14x14mm_P0.5mm, symbol MCU_ST_STM32F4:STM32F405VGTx
- removed U9: LTC4412xS6, Package_TO_SOT_SMD:TSOT-23-6, symbol Power_Management:LTC4412xS6
- removed UMMC5983MA: ~, symbol MMC5983ma_Ray:MMC5983ma
- added 5k1: 10k, symbol Device:R
- added BZ1: Active Buzzer, symbol Device:Buzzer
- added C35, C36: 100n, symbol Device:C
- added D11: R, symbol Device:LED
- added D12: 1N4148, Diode_THT:D_DO-35_SOD27_P7.62mm_Horizontal, symbol Diode:1N4148
- added D2: B_3V3, symbol Device:LED
- added D3: TVS, symbol Device:D_TVS_Filled
- added D8: G, symbol Device:LED
- added J10, J12: Conn_01x04, symbol Connector_Generic:Conn_01x04
- added J4: Conn_01x03, symbol Connector_Generic:Conn_01x03
- added J6: Screw_Terminal_01x01, symbol Connector:Screw_Terminal_01x01
- added Q1, Q2: TSM3481CX6 RFG, Package_TO_SOT_SMD:SOT-23, symbol Transistor_FET:IRLML6402
- added Q5: NMOS, symbol Simulation_SPICE:NMOS
- added R43: 390k, symbol Device:R
- added SW2: USER_Buttom, symbol Switch:SW_Push
- added U2: LD1117S33TR_SOT223, Package_TO_SOT_SMD:SOT-223-3_TabPin2, symbol Regulator_Linear:LD1117S33TR_SOT223
- added U3: LTC4412xS6, Package_TO_SOT_SMD:TSOT-23-6, symbol Power_Management:LTC4412xS6
- added U4: TPS54538RQFR, VQFN-HR9_RQF_TEX, symbol Small_av_tony_lib:TPS54538RQFR
- added U5: BMI088, Package_LGA:Bosch_LGA-16_4.5x3mm_P0.5mm_LayoutBorder7x1y_ClockwisePinNumbering, symbol Sensor_Motion:BMI088
- added U6: BMP390, 10LGA_2X2X0p75_BOS, symbol Small_av_tony_lib:BMP390
- added U7: MMC5983MA, MMC5983MA_MEM, symbol Small_av_tony_lib:MMC5983MA
- added U8: W25Q128JVS, Package_SO:SOIC-8_5.3x5.3mm_P1.27mm, symbol Memory_Flash:W25Q128JVS
- C1, C2, C3, C4, C6: value C -> 100n
- C10, C11: value 10uF -> 22pF
- C12, C9: value 10uF -> 100n
- C13, C14, C15: value 10uF -> 4.7u
- C20: value 4.7u -> 100n
- C27: value 10u -> 100n
- C28: value 1n -> 1u
- C29: value 22pF -> 10u
- C30: value 22pF -> 1u
- C31: value 100nF -> 4.7u
- C32: value 100nF -> 100n
- C5: value C -> 10u
- C7: value C -> 1u
- D1: value LED -> G_5V
- L1: value L -> 6.8u
- R1, R2: value 4.7K -> 10k
- R13: value 1K -> 18k
- R14: value 2.2k -> 220k
- R15: value 2.2k -> 30k
- R16, R17: value 4.7K -> 1k
- R18, R19, R21: value 4.7K -> 100k
- R20: value 4.7K -> 1M
- R24, R25: value 22ohm -> 2.7k
- R28: value 100k -> 10k
- R29: value 18k -> 10k
- R3: value 4.7K -> 0 ohm
- R35: value 0 ohm -> 2.2k
- R38: value 1k -> 2.2k
- R4: value 4.7K -> 22ohm
- R40: value 1.5k -> 10k
- R41: value 5.1k -> 10k
- R42: value 5.1k -> 100k
- R5: value 10K -> 22ohm
- R6, R7: value 10K -> 5.1k
- R8: value 10K -> 1.5k
- renumbered Buck_5v to Buck_5v1, GND to GND2, R16(PG_pull_up) to R16(PG_pull_up)1, V_BAT+ to V_BAT+1
Connections:
- net +3V3 is gone; now on net +3.3V: C1.1, C3.1
- net CAP is gone; now on net HSE_IN: C10.1
- net IO3/Hold is gone; now on net BUCK_5V: R16.2
- net MOSI is gone; now on net GND: R6.2
- net SCK is gone; now on net +3.3V: R8.2
- net SCL_3v3 is gone; now on net GND: R2.2
- net +3.3V: now also C2.1, C20.1, C25.1, C26.1, C27.1, C28.1, C30.1, C31.1, C32.1, C4.1, C5.1, FB1.2, R17.2, R21.1, R22.2, R23.2, R24.1, R25.1, R26.2, R27.2, R28.1, R29.2, J12.3 (Pin_3), U2.2 (VO), U5.11 (VDDIO), U5.3 (VDD), U6.1 (VDDIO), U6.10 (VDD), U7.13 (VDDIO), U7.2 (VDD), U7.4 (SPI_CS), U8.8 (VCC); no longer R26.1, R39.2, R40.2
- net +USB_5V: now also R19.2, Q2.3 (D), U3.6 (SENSE)
- net BOOT0: now also R1.1; no longer R23.1
- net BOOT1: now also R2.1; no longer R22.1
- net BUCK_5V: now also L1.1, R14.1, Q2.2 (S), U2.3 (VI), U3.1 (VIN); no longer R38.2
- net HSE_IN: no longer C29.1
- net HSE_OUT: now also R3.1; no longer R35.1
- net I2C1_SCL: now also R24.2, U1.42 (PB6), J12.1 (Pin_1), U7.1 (SCL/SPI_SCK)
- net I2C1_SDA: now also R25.2, U1.43 (PB7), J12.2 (Pin_2), U7.16 (SDA/SPI_SDI)
- net PG_BUCK: now also U4.9 (SS/PG)
- net RST: now also C9.1
- net SPI1_MISO: now also U1.16 (PA6), U5.10 (SDO2), U5.15 (SDO1), U6.5 (SDO)
- net SPI1_MOSI: now also U1.17 (PA7), U5.9 (SDI/SDA), U6.4 (SDI)
- net SPI1_SCK: now also U1.15 (PA5), U5.8 (SCK/SCL), U6.2 (SCK)
- net SUP_STAT: now also R21.2, U3.4 (STAT)
- net SWCLK: now also J3.3 (Pin_3); no longer R25.1
- net SWDIO: now also J3.2 (Pin_2); no longer R24.1
- net USB_D+: now also R5.1, R8.1; no longer R40.1
- net USB_D-: now also R4.2
- net V_BAT+: now also C12.1, C13.1, C14.1, C15.1, R41.2, BZ1.1 (+), D12.1 (K), Q1.2 (S), R43.2, U4.5 (VIN), U4.6 (VIN); no longer C20.1, C25.1
- net at C16.2: now also R14.2, R15.1, U4.3 (FB)
- net at R39.1: now also R40.1, Q5.2 (G)
- net at C6.1, C7.1: now also FB1.1, U1.9 (VDDA)
- net at R16.1: now also D1.2 (A); no longer R17.1
- net CSB_Flash: now reaches R29.1
- net CSB_Flash: now also U1.29 (PA8), U8.1 (~{CS})
- net at F1.2: now also D3.2 (A2), Q1.3 (D)
- net at J2.A5 (CC1): now also R6.1; no longer R41.1
- net at J2.A6 (D+), J2.B6 (D+): now also R5.2
- net at J2.A7 (D-), J2.B7 (D-): now also R4.1
- net at J2.B5 (CC2): now also R7.1; no longer R42.1
- net at R19.1, R20.1: now also U3.3 (CTL); no longer R18.1
- net GND: now reaches C4.2
- net GND: now also C1.2, C10.2, C11.2, C12.2, C13.2, C14.2, C15.2, C17.2, C18.2, C19.2, C2.2, C20.2, C21.2, C22.2, C23.2, C24.2, C25.2, C26.2, C27.2, C28.2, C29.2, C3.2, C30.2, C31.2, C32.2, C5.2, C6.2, C7.2, C9.2, D1.1 (K), GND2.1, J2.A1 (GND), J2.A12 (GND), J2.B1 (GND), J2.B12 (GND), J2.S1 (SHIELD), J3.4 (Pin_4), J5.2 (Pin_2), R1.2, R13.2, R15.2, R18.2, R20.2, R35.1, R38.1, R40.2, R42.1, R7.2, SW1.1, U1.23 (VSS), U1.35 (VSS), U1.47 (VSS), U1.8 (VSSA), Y1.2 (G), Y1.4 (G), 5k1.1, C35.2, C36.2, D2.1 (K), D3.1 (A1), J10.3 (Pin_3), J10.4 (Pin_4), J12.4 (Pin_4), J4.3 (Pin_3), J6.1 (Pin_1), Q5.3 (S), SW2.1, U2.1 (GND), U3.2 (GND), U4.4 (GND), U5.2 (GNDA), U5.4 (GNDA), U5.6 (GNDIO), U5.7 (PS), U6.3 (VSS), U6.8 (VSS), U6.9 (VSS), U7.11 (GND), U7.9 (GND), U8.4 (GND)
- net at R35.2: now also D8.1 (K); no longer C30.1
- net INT_Accel1: now reaches U1.10 (PA0)
- net INT_Accel1: now also U5.16 (INT1)
- net INT_Accel2: now reaches U1.11 (PA1)
- net INT_Accel2: now also U5.1 (INT2)
- net INT_Gyro: now reaches U1.12 (PA2)
- net INT_Gyro: now also U5.12 (INT3)
- net CSB_Gyro: now reaches U1.13 (PA3)
- net CSB_Gyro: now also R23.1, U5.5 (~{CSB2})
- net CSB_Accel: now reaches U1.14 (PA4)
- net CSB_Accel: now also R22.1, U5.14 (~{CSB1})
- net CSB_Baro: now reaches U1.18 (PB0)
- net CSB_Baro: now also R28.2, U6.6 (CSB)
- net Battery_Sensing: now reaches U1.19 (PB1)
- net Battery_Sensing: now also R41.1, 5k1.2, C35.1
- net LED_SYS: now reaches U1.2 (PC13)
- net LED_SYS: now also D8.2 (A)
- net INT_Baro: now reaches U1.21 (PB10)
- net INT_Baro: now also U6.7 (INT)
- net Buzzer: now reaches U1.22 (PB11)
- net Buzzer: now also R39.2
- net WP_Flash: now reaches U1.25 (PB12)
- net WP_Flash: now also R27.1, U8.3 (~{WP}/IO_{2})
- net SPI2_SCK: now reaches U1.26 (PB13)
- net SPI2_SCK: now also U8.6 (CLK)
- net SPI2_MISO: now reaches U1.27 (PB14)
- net SPI2_MISO: now also U8.2 (DO/IO_{1})
- net SPI2_MOSI: now reaches U1.28 (PB15)
- net SPI2_MOSI: now also U8.5 (DI/IO_{0})
- net LED_State: now reaches U1.3 (PC14)
- net LED_State: now also D11.2 (A)
- net USART1_TX: now reaches U1.30 (PA9)
- net USART1_TX: now also J4.1 (Pin_1)
- net USART1_RX: now reaches U1.31 (PA10)
- net USART1_RX: now also J4.2 (Pin_2)
- net USER_BT: now reaches U1.4 (PC15)
- net USER_BT: now also C36.1, SW2.2
- net INT_Magn: now reaches U1.41 (PB5)
- net INT_Magn: now also U7.15 (INT)
- net FIRE: now reaches U1.45 (PB8)
- net FIRE: now also J10.2 (Pin_2)
- net PWM Servo: now reaches U1.46 (PB9)
- net PWM Servo: now also J10.1 (Pin_1)
- removed net +3.3VA: C26.1, C27.1, FB1.1, U1.9 (VDDA)
- removed net 3v3: C1.2, C10.2, C11.1, C11.2, C12.1, C12.2, C13.1, C13.2, C14.2, C15.2, C17.2, C18.2, C19.2, C2.1, C2.2, C20.2, C21.2, C22.2, C23.2, C24.2, C25.2, C26.2, C27.2, C28.2, C29.2, C3.2, C30.2, C31.1, C31.2, C32.1, C32.2, C5.1, C5.2, C6.2, C7.2, C9.1, C9.2, D1.1 (K), GND2.1, J2.A1 (GND), J2.A12 (GND), J2.B1 (GND), J2.B12 (GND), J2.S1 (SHIELD), J3.4 (Pin_4), J5.2 (Pin_2), R1.1, R13.1, R17.2, R18.2, R20.2, R22.2, R23.2, R27.2, R28.2, R29.2, R4.1, R41.2, R42.2, R5.1, R6.1, R7.1, R8.1, SW1.1, U1.23 (VSS), U1.35 (VSS), U1.47 (VSS), U1.8 (VSSA), Y1.2 (G), Y1.4 (G)
- removed net CS: R19.2, R7.2
- removed net SCL: R1.2, R14.2, R15.2, R2.1, R3.1, R4.2
- net SDA_3v3: no longer names the net of R3.2
- net SDA_3v3: now also C11.1
- new net: R26.1, U8.7 (~{HOLD}/~{RESET}/IO_{3})
- new net: C29.1, U7.10 (CAP)
- new net: BZ1.2 (-), D12.2 (A), Q5.1 (D)
- new net: D11.1 (K), R38.2
- new net: Q2.1 (G), U3.5 (GATE)
- new net: R42.2, R43.1, U4.2 (EN)
- new net: L1.2, U4.8 (SW)
- new net: R13.1, U4.7 (MODE)
- new net: D2.2 (A), R17.1
- new net: Q1.1 (G), R18.1
- no-connect marks 5 -> 4
Other:
- note added: "Barometer"
- note added: "Battery monitor"
- note added: "Buttom"
- note added: "Connection to Main_AV"
- note added: "Flash"
- note added: "IMU"
- note added: "Ignition connector"
- note added: "Magnetometer"
- note added: "Power management"
- note added: "Reserved connector"
- note added: "UART communication"
- note added: "common ground to Main_AV GND"
- note added: "decoupling for VDD,VDDIO"
- note added: "maybe a remove before flight?"
- note removed: "+"
- note removed: "-"
- note removed: "Barometer - BMP390"
- note removed: "Connectors"
- note removed: "Jumpers"
- note removed: "LEVEL SHIFTING (5V <--> 3V)"
- note removed: "MMC5983MA_QFN16"
- note removed: "Magnetometer - MMC5983MA_QFN16"
- note removed: "NOR Flash"
- note removed: "Power 模組"
- note removed: "QWIC_RIGHT_ANGLE"
- note removed: "TP1"
- note removed: "TP2"
- note removed: "TP3"
- note removed: "TP5"
- note removed: "Testpoint"
- note removed: "VDD 2.8~3.6 V VDDIO 2.8~3.6V I2C address : 0x30"
- note removed: "cut trace to disconnect Power LED"
- note removed: "cut trace to remove I2C pull-up resistors"
- note removed: "lout"
- note removed: "Ｆor SOI set CSB low at startup DD=MISO, SDI=MOSI,SCK=SCK, CSB=CS/SSEL For IC leave CSB pulled high (default value) SDI=SDA, SCK=SCL"
- moved on the sheet: 3V3, Buck_5v1, C16, C17, C18, C19, C21, C22, C23, C24, F1, FB1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
