File: SmallAvionic/Tony/SmallAvionic.kicad_sch (KiCad schematic)
At the start: 103 parts, among them J1 Boot_mode_pin, J10 Conn_01x04, J2 USB_C_Receptacle_USB2.0_16P, J3 Conn_01x04, J4 Conn_01x03, J5 Conn_01x02, J6 Screw_Terminal_01x01, Q1 TSM3481CX6 RFG, Q2 TSM3481CX6 RFG, Q5 NMOS, SW1 SW_Push, U1 STM32F103C8Tx, U2 LD1117S33TR_SOT223, U3 LTC4412xS6, U4 TPS54538RQFR, U5 BMI088, U6 BMP390, U7 MMC5983MA, U8 W25Q128JVS, Y1 8Mhz

Commit message: slight modification on small AV , start Big AV
Parts:
- removed C8: 1n, symbol Device:C
- added C36: 100n, symbol Device:C
- added J12: Conn_01x04, symbol Connector_Generic:Conn_01x04
- added R42: 100k, symbol Device:R
- added R43: 390k, symbol Device:R
- added SW2: USER_Buttom, symbol Switch:SW_Push
- C7: value 10u -> 1u
Connections:
- net +3.3V: now also FB1.2, J12.3 (Pin_3); no longer C6.1, C7.1, FB1.1, U1.9 (VDDA)
- net GND: now also C36.2, J12.4 (Pin_4), R42.1, SW2.1
- net I2C1_SCL: now also J12.1 (Pin_1)
- net I2C1_SDA: now also J12.2 (Pin_2)
- net V_BAT+: now also R43.2
- net USER_BT: now reaches U1.4 (PC15)
- net USER_BT: now also C36.1, SW2.2
- net V_BAT: no longer names the net of U4.2 (EN)
- net V_BAT: now also R42.2, R43.1
- new net: C6.1, C7.1, FB1.1, U1.9 (VDDA)
Other:
- note added: "Buttom"
- note added: "Reserved connector"
- note added: "maybe a remove before flight?"
- moved on the sheet: BZ1, D11, D12, D8, J10, Q5, R35, R38, R39, R40
