File: BigAvionic/Iusbubula_Avionic_Board.kicad_sch (KiCad schematic)
At the start: 38 parts, among them J5 Conn_01x02, Q1 TSM3481CX6 RFG, Q2 TSM3481CX6 RFG, U1 STM32F405VGTx, U2 LD1117S33TR_SOT223, U3 LTC4412xS6, U4 TPS54538RQFR

Commit message: fix autosave problem
Parts:
- added C1, C2: 2.2u, symbol Device:C
- added C10: 10u, symbol Device:C
- added C11: 1u, symbol Device:C
- added C20: 1n, symbol Device:C
- added C25, C3, C4, C5, C6, C7, C8, C9: 100n, symbol Device:C
- added FB1: FerriteBead 120R @ 100M, symbol Device:FerriteBead
- added R1: 390k, symbol Device:R
- added R2: 100k, symbol Device:R
Connections:
- net GND: now also C1.2, C10.2, C11.2, C2.2, C20.2, C25.2, C3.2, C4.2, C5.2, C6.2, C7.2, C8.2, C9.2, R2.1
- net V_BAT+: now also R1.2
- net +3V3: now reaches U1.100 (VDD)
- net +3V3: now also U1.11 (VDD), U1.19 (VDD), U1.28 (VDD), U1.50 (VDD), U1.6 (VBAT), U1.75 (VDD), C10.1, C3.1, C4.1, C5.1, C6.1, C7.1, C8.1, C9.1, FB1.2
- net VREF: now reaches U1.22 (VDDA)
- net VREF: now also C11.1, C20.1, C25.1, FB1.1
- net at U1.49 (VCAP_1): now also C2.1
- net at U1.73 (VCAP_2): now also C1.1
- net V_BAT: no longer names the net of U4.2 (EN)
- net V_BAT: now also R1.1, R2.2
Other:
- note added: "ESR<2ohm"
