File: BigAvionic/Iusbubula_Avionic_Board.kicad_sch (KiCad schematic)
At the start: 156 parts, among them J1 Conn_01x02, J10 Conn_01x04, J12 Conn_01x04, J2 USB_C_Receptacle_USB2.0_16P, J3 Conn_01x04, J4 Conn_Coaxial, J5 Conn_01x02, J6 Micro_SD_Card_Det1, J7 Screw_Terminal_01x01, J8 Conn_01x03, Q1 TSM3481CX6 RFG, Q2 TSM3481CX6 RFG, Q5 NMOS, SW1 SW_Push, SW2 USER_Buttom, SW3 USER_Buttom, U1 STM32F405VGTx, U10 E22-400T30S, U11 E80-900M23313S, U12 W25Q128JVS, U2 LD1117S33TR_SOT223, U3 LTC4412xS6, U4 TPS54538RQFR, U5 BMI088, U6 BMP390, U7 MMC5983MA, U8 ADXL375BCCZ, U9 NEO-M9N-00B, Y1 8Mhz

Commit message: check
Parts:
- removed 5k: 10k, symbol Device:R
- removed J8: Conn_01x03, symbol Connector_Generic:Conn_01x03
- removed R5: 0ohm, symbol Device:R
- added J9: Conn_01x04, Connector_JST:JST_EH_S4B-EH_1x04_P2.50mm_Horizontal, symbol Connector_Generic:Conn_01x04
- added R54: 0ohm, symbol Device:R
- added R55: 5k, symbol Device:R
- 3V3: footprint (none) -> TestPoint:TestPoint_Pad_D1.0mm
- BZ1: footprint (none) -> Buzzer_Beeper:Buzzer_12x9.5RM7.6
- Buck_5v1: renamed from Buck_5v; footprint (none) -> TestPoint:TestPoint_Pad_D1.0mm
- C1, C10, C11, C12, C13, C14, C15, C16, C17, C18, C19, C2, C20, C21, C22, C23, C24, C25, C26, C27, C28, C29, C3, C30, C31, C32, C33, C34, C35, C36, C37, C38, C39, C4, C40, C41, C42, C43, C44, C45, C46, C47, C48, C49, C5, C50, C51, C52, C53, C6, C7, C8, C9: footprint (none) -> Capacitor_SMD:C_0805_2012Metric_Pad1.18x1.45mm_HandSolder
- D1, D11, D2, D3, D4, D5, D8: footprint (none) -> LED_SMD:LED_0805_2012Metric_Pad1.15x1.40mm_HandSolder
- D12: footprint Diode_THT:D_DO-35_SOD27_P7.62mm_Horizontal -> LED_SMD:LED_0805_2012Metric_Pad1.15x1.40mm_HandSolder
- F1: footprint (none) -> Fuse:Fuse_0805_2012Metric_Pad1.15x1.40mm_HandSolder
- FB1: footprint (none) -> Inductor_SMD:L_0805_2012Metric_Pad1.05x1.20mm_HandSolder
- GND1: renamed from GND; footprint (none) -> TestPoint:TestPoint_Pad_1.0x1.0mm
- J1: footprint (none) -> Connector_PinHeader_2.54mm:PinHeader_1x02_P2.54mm_Vertical
- J10: footprint (none) -> Connector_JST:JST_EH_S4B-EH_1x04_P2.50mm_Horizontal
- J12: footprint (none) -> Connector_JST:JST_EH_B4B-EH-A_1x04_P2.50mm_Vertical
- J2: footprint (none) -> Connector_USB:USB_C_Receptacle_HRO_TYPE-C-31-M-12
- J3: footprint (none) -> Connector_PinHeader_2.54mm:PinHeader_1x04_P2.54mm_Vertical
- J4: footprint (none) -> Connector_Coaxial:U.FL_Hirose_U.FL-R-SMT-1_Vertical
- J5: footprint (none) -> Connector_JST:JST_PH_S2B-PH-K_1x02_P2.00mm_Horizontal
- J6: footprint (none) -> Connector_Card:microSD_HC_Molex_47219-2001
- J7: footprint (none) -> TerminalBlock_Phoenix:TerminalBlock_Phoenix_PT-1,5-2-3.5-H_1x02_P3.50mm_Horizontal
- U4: footprint VQFN-HR9_RQF_TEX -> (none)
- U6: footprint 10LGA_2X2X0p75_BOS -> (none)
- U7: footprint MMC5983MA_MEM -> (none)
- U8: footprint LGA_CC-14-1_ADI -> (none)
- U9: footprint SMT_9N-00B_UBL -> (none)
- renumbered R16(PG_pull_up) to R16(PG_pull_up)1, V_BAT+ to V_BAT+1
Connections:
- net Battery_Sensing: now also R55.2
- net GND: now also J9.3 (Pin_3), R55.1
- net USART2_RX: now also J9.1 (Pin_1)
- net USART2_TX: now also J9.2 (Pin_2)
- net USB_D+: now also R54.2
- net at J2.A6 (D+), J2.B6 (D+): now also R54.1
- net RST renamed RESET
- net RESET: now also J9.4 (Pin_4)
- no-connect marks 26 -> 46

Commit message: slight modification
Parts:
- removed L2: short, symbol Device:L
- removed R27: NC, symbol Device:R
Connections:
- net at C41.1, C42.1: now also J4.1 (In)
- no-connect marks 46 -> 47
Other:
- note removed: "Reserved for active atenna"
- moved on the sheet: C41
Changed lines of the file:
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@@
 		)
 	)
-	(text "Reserved for active atenna"
-		(exclude_from_sim no)
-		(at 365.252 136.652 0)
-		(effects
-			(font
-				(size 1.27 1.27)
-			)
-		)
-	)
 	(text "High g accel meter\n"
 		(exclude_from_sim no)
@@
 	)
 	(junction
-		(at 53.34 114.3)
+		(at 364.49 132.08)
 		(diameter 0)
 		(color 0 0 0 0)
 	)
 	(junction
-		(at 92.71 317.5)
+		(at 53.34 114.3)
 		(diameter 0)
 		(color 0 0 0 0)
 	)
 	(junction
-		(at 41.91 71.12)
+		(at 92.71 317.5)
 		(diameter 0)
 		(color 0 0 0 0)
 	)
 	(junction
-		(at 363.22 124.46)
+		(at 41.91 71.12)
 		(diameter 0)
 		(color 0 0 0 0)
@@
 	)
 	(junction
-		(at 365.76 132.08)
-		(diameter 0)
-		(color 0 0 0 0)
-	)
-	(junction
 		(at 162.56 34.29)
 		(diameter 0)
@@
 	)
 	(junction
+		(at 364.49 124.46)
+		(diameter 0)
+		(color 0 0 0 0)
+	)
+	(junction
 		(at 257.81 156.21)
 		(diameter 0)
@@
 	)
 	(junction
-		(at 365.76 124.46)
-		(diameter 0)
-		(color 0 0 0 0)
-	)
-	(junction
 		(at 356.87 227.33)
 		(diameter 0)
@@
 	)
 	(no_connect
+		(at 374.65 119.38)
+	)
+	(no_connect
 		(at 148.59 152.4)
 	)
@@
 	(wire
 		(pts
+			(xy 364.49 132.08) (xy 374.65 132.08)
+		)
+		(stroke
+			(width 0)
+			(type default)
+		)
+	)
+	(wire
+		(pts
 			(xy 316.23 339.09) (xy 323.85 339.09)
 		)
@@
 	(wire
 		(pts
+			(xy 364.49 124.46) (xy 365.76 124.46)
+		)
+		(stroke
+			(width 0)
+			(type default)
+		)
+	)
+	(wire
+		(pts
 			(xy 120.65 34.29) (xy 123.19 34.29)
 		)
@@
 	(wire
 		(pts
-			(xy 349.25 132.08) (xy 365.76 132.08)
+			(xy 349.25 132.08) (xy 364.49 132.08)
 		)
 		(stroke
@@
 	(wire
 		(pts
-			(xy 363.22 119.38) (xy 363.22 124.46)
-		)
-		(stroke
-			(width 0)
-			(type default)
-		)
-	)
-	(wire
-		(pts
 			(xy 378.46 46.99) (xy 369.57 46.99)
 		)
@@
 	(wire
 		(pts
-			(xy 365.76 132.08) (xy 374.65 132.08)
-		)
-		(stroke
-			(width 0)
-			(type default)
-		)
-	)
-	(wire
-		(pts
 			(xy 280.67 347.98) (xy 279.4 347.98)
 		)
@@
 	(wire
 		(pts
-			(xy 363.22 124.46) (xy 365.76 124.46)
-		)
-		(stroke
-			(width 0)
-			(type default)
-		)
-	)
-	(wire
-		(pts
 			(xy 115.57 346.71) (xy 115.57 359.41)
 		)
@@
 	(wire
 		(pts
-			(xy 370.84 119.38) (xy 374.65 119.38)
-		)
-		(stroke
-			(width 0)
-			(type default)
-		)
-	)
-	(wire
-		(pts
 			(xy 105.41 364.49) (xy 106.68 364.49)
 		)
@@
 	(wire
 		(pts
-			(xy 354.33 124.46) (xy 355.6 124.46)
+			(xy 354.33 124.46) (xy 364.49 124.46)
 		)
 		(stroke
@@
 	(symbol
 		(lib_id "Device:C")
-		(at 365.76 128.27 0)
+		(at 364.49 128.27 0)
 		(mirror y)
 		(unit 1)
@@
 		(dnp no)
 		(property "Reference" "C41"
-			(at 362.712 126.746 0)
+			(at 361.442 126.746 0)
 			(effects
 				(font
@@
 		)
 		(property "Value" "NC"
-			(at 362.712 129.5399 0)
+			(at 361.442 129.5399 0)
 			(effects
 				(font
@@
 		)
 		(property "Footprint" "Capacitor_SMD:C_0805_2012Metric_Pad1.18x1.45mm_HandSolder"
-			(at 364.7948 132.08 0)
+			(at 363.5248 132.08 0)
 			(effects
 				(font
@@
 		)
 		(property "Datasheet" "~"
-			(at 365.76 128.27 0)
+			(at 364.49 128.27 0)
 			(effects
 				(font
@@
 		)
 		(property "Description" "Unpolarized capacitor"
-			(at 365.76 128.27 0)
+			(at 364.49 128.27 0)
 			(effects
 				(font
@@
 	)
 	(symbol
-		(lib_id "Device:L")
-		(at 359.41 124.46 90)
-		(unit 1)
-		(exclude_from_sim no)
-		(in_bom yes)
-		(on_board yes)
-		(dnp no)
-		(fields_autoplaced yes)
-		(property "Reference" "L2"
-			(at 359.41 119.38 90)
-			(effects
-				(font
-					(size 1.27 1.27)
-				)
-			)
-		)
-		(property "Value" "short"
-			(at 359.41 121.92 90)
-			(effects
-				(font
-					(size 1.27 1.27)
-				)
-			)
-		)
-		(property "Footprint" ""
-			(at 359.41 124.46 0)
-			(effects
-				(font
-					(size 1.27 1.27)
-				)
-				(hide yes)
-			)
-		)
-		(property "Datasheet" "~"
-			(at 359.41 124.46 0)
-			(effects
-				(font
-					(size 1.27 1.27)
-				)
-				(hide yes)
-			)
-		)
-		(property "Description" "Inductor"
-			(at 359.41 124.46 0)
-			(effects
-				(font
-					(size 1.27 1.27)
-				)
-				(hide yes)
-			)
-		)
-		(pin "1"
-		)
-		(pin "2"
-		)
-		(instances
-			(project ""
-				(path "/80a059dc-2311-4dd3-afad-18a5367fc218"
-					(reference "L2")
-					(unit 1)
-				)
-			)
-		)
-	)
-	(symbol
 		(lib_id "Connector_Generic:Conn_01x04")
 		(at 281.94 306.07 0)
@@
 					(unit 1)
 				)
-			)
-		)
-	)
-	(symbol
-		(lib_id "Device:R")
-		(at 367.03 119.38 90)
-		(mirror x)
-		(unit 1)
-		(exclude_from_sim no)
-		(in_bom yes)
-		(on_board yes)
-		(dnp no)
-		(property "Reference" "R27"
-			(at 364.744 113.03 90)
-			(effects
-				(font
-					(size 1.27 1.27)
-				)
-				(justify left)
-			)
-		)
-		(property "Value" "NC"
-			(at 364.236 115.57 90)
-			(effects
-				(font
-					(size 1.27 1.27)
-				)
-				(justify left)
-			)
-		)
-		(property "Footprint" ""
-			(at 367.03 117.602 90)
-			(effects
-				(font
-					(size 1.27 1.27)
-				)
-				(hide yes)
-			)
-		)
-		(property "Datasheet" "~"
-			(at 367.03 119.38 0)
-			(effects
-				(font
-					(size 1.27 1.27)
-				)
-				(hide yes)
-			)
-		)
-		(property "Description" "Resistor"
-			(at 367.03 119.38 0)
-			(effects
-				(font
-					(size 1.27 1.27)
-				)
-				(hide yes)
-			)
-		)
-		(pin "2"
-		)
-		(pin "1"
-		)
-		(instances
-			(project "Iusbubula_Avionic_Board"
-				(path "/80a059dc-2311-4dd3-afad-18a5367fc218"
-					(reference "R27")
-					(unit 1)
-				)
