File: BigAvionic/Iusbubula_Avionic_Board.kicad_sch (KiCad schematic)
At the start: 137 parts, among them J1 Conn_01x02, J10 Conn_01x04, J12 Conn_01x04, J2 USB_C_Receptacle_USB2.0_16P, J3 Conn_01x04, J5 Conn_01x02, J6 Micro_SD_Card_Det1, J7 Screw_Terminal_01x01, J9 Conn_01x04, Q1 TSM3481CX6 RFG, Q2 TSM3481CX6 RFG, Q5 NMOS, SW1 SW_Push, SW2 USER_Buttom, SW3 USER_Buttom, U1 STM32F405VGTx, U10 E22-400T30S, U11 E80-900M23313S, U12 W25Q128JVS, U2 LD1117S33TR_SOT223, U3 LTC4412xS6, U4 TPS54538RQFR, U5 BMI088, U6 BMP390, U8 ADXL375BCCZ, Y1 8Mhz

Commit message: finish power layer(still need check)
Parts:
- removed C1, C2: 2.2u, Capacitor_SMD:C_0805_2012Metric_Pad1.18x1.45mm_HandSolder, symbol Device:C
- removed C10, C38, C47: 10u, Capacitor_SMD:C_0805_2012Metric_Pad1.18x1.45mm_HandSolder, symbol Device:C
- removed C11: 1u, Capacitor_SMD:C_0805_2012Metric_Pad1.18x1.45mm_HandSolder, symbol Device:C
- removed C20: 1n, Capacitor_SMD:C_0805_2012Metric_Pad1.18x1.45mm_HandSolder, symbol Device:C
- removed C25, C26, C29, C3, C30, C31, C32, C36, C37, C4, C48, C5, C50, C6, C7, C8, C9: 100n, Capacitor_SMD:C_0805_2012Metric_Pad1.18x1.45mm_HandSolder, symbol Device:C
- removed C27, C28: 22pF, Capacitor_SMD:C_0805_2012Metric_Pad1.18x1.45mm_HandSolder, symbol Device:C
- removed C49: 4.7u, Capacitor_SMD:C_0805_2012Metric_Pad1.18x1.45mm_HandSolder, symbol Device:C
- removed FB1: FerriteBead 120R @ 100M, Inductor_SMD:L_0805_2012Metric_Pad1.05x1.20mm_HandSolder, symbol Device:FerriteBead
- removed J1: Conn_01x02, Connector_PinHeader_2.54mm:PinHeader_1x02_P2.54mm_Vertical, symbol Connector_Generic:Conn_01x02
- removed J2: USB_C_Receptacle_USB2.0_16P, Connector_USB:USB_C_Receptacle_HRO_TYPE-C-31-M-12, symbol Connector:USB_C_Receptacle_USB2.0_16P
- removed J3: Conn_01x04, Connector_PinHeader_2.54mm:PinHeader_1x04_P2.54mm_Vertical, symbol Connector_Generic:Conn_01x04
- removed J6: Micro_SD_Card_Det1, Connector_Card:microSD_HC_Molex_47219-2001, symbol Connector:Micro_SD_Card_Det1
- removed R10: 0 ohm, Resistor_SMD:R_0805_2012Metric_Pad1.20x1.40mm_HandSolder, symbol Device:R
- removed R22, R23, R28, R3, R4, R45, R46, R47, R8, R9: 10k, Resistor_SMD:R_0805_2012Metric_Pad1.20x1.40mm_HandSolder, symbol Device:R
- removed R27, R34, R36, R37, R39, R42, R43: 22ohm, Resistor_SMD:R_0805_2012Metric_Pad1.20x1.40mm_HandSolder, symbol Device:R
- removed R35, R38, R40, R41, R44: 47k, Resistor_SMD:R_0805_2012Metric_Pad1.20x1.40mm_HandSolder, symbol Device:R
- removed R5, R54: 0ohm, Resistor_SMD:R_0805_2012Metric_Pad1.20x1.40mm_HandSolder, symbol Device:R
- removed R6, R7: 5.1k, Resistor_SMD:R_0805_2012Metric_Pad1.20x1.40mm_HandSolder, symbol Device:R
- removed SW1: SW_Push, Button_Switch_THT:SW_PUSH_6mm_H4.3mm, symbol Switch:SW_Push
- removed U1: STM32F405VGTx, Package_QFP:LQFP-100_14x14mm_P0.5mm, symbol MCU_ST_STM32F4:STM32F405VGTx
- removed U12: W25Q128JVS, Package_SO:SOIC-8_5.3x5.3mm_P1.27mm, symbol Memory_Flash:W25Q128JVS
- removed U5: BMI088, Package_LGA:Bosch_LGA-16_4.5x3mm_P0.5mm_LayoutBorder7x1y_ClockwisePinNumbering, symbol Sensor_Motion:BMI088
- removed U6: BMP390, Tony:10LGA_2X2X0p75_BOS-M, symbol Small_av_tony_lib:BMP390
- removed U8: ADXL375BCCZ, Tony:LGA_CC-14-1_ADI-L, symbol A_library:ADXL375BCCZ
- removed Y1: 8Mhz, Crystal:Crystal_HC49-U_Vertical, symbol Device:Crystal_GND24
Connections:
- no-connect marks 34 -> 9
Other:
- note removed: "Barometer"
- note removed: "ESR<2ohm"
- note removed: "External reset"
- note removed: "Flash"
- note removed: "HSE crystal"
- note removed: "High g accel meter"
- note removed: "IMU"
- note removed: "MCU"
- note removed: "SD card"
- note removed: "Serial Wire Debug"
- note removed: "USB"
- note removed: "boot mode"
- note removed: "decoupling"
- note removed: "decoupling for VDD,VDDIO"
