File: GroundStation/GroundStation/GroundStation.kicad_pcb (KiCad board)
At the start: 4 copper layers, 83 x 108.3 mm, 72 parts, among them J1 SD_Card_Receptacle, J4 Conn_Coaxial, J5 Conn_01x02, P1 USB_C_Plug_USB2.0, Q1 TSM3481CX6 RFG, U1 STM32F103C8Tx, U10 E22-400T30S, U101 LD1117S33TR_SOT223, U11 E80-900M23313S, U4 TPS54538RQFR, U9 NEO-M9N-00B

Commit message: 4/20grounglast
Parts:
- removed C12: 100n, Capacitor_SMD:C_0805_2012Metric_Pad1.18x1.45mm_HandSolder
- removed C13, C14, C15: 4.7u, Capacitor_SMD:C_0805_2012Metric_Pad1.18x1.45mm_HandSolder
- removed C16: 10p, Capacitor_SMD:C_0805_2012Metric_Pad1.18x1.45mm_HandSolder
- removed C17, C18, C19: 47u, Capacitor_SMD:C_0805_2012Metric_Pad1.18x1.45mm_HandSolder
- removed C41: NC, Capacitor_SMD:C_0805_2012Metric_Pad1.18x1.45mm_HandSolder
- removed C42: 100p, Capacitor_SMD:C_0805_2012Metric_Pad1.18x1.45mm_HandSolder
- removed D103: TVS, Diode_SMD:D_SOD-123
- removed L1: 6.8u, Inductor_SMD:L_0805_2012Metric_Pad1.05x1.20mm_HandSolder
- removed L2: short, Inductor_SMD:L_Bourns_SDR0604
- removed R1: 390k, Resistor_SMD:R_0805_2012Metric_Pad1.20x1.40mm_HandSolder
- removed R13: 18k, Resistor_SMD:R_0805_2012Metric_Pad1.20x1.40mm_HandSolder
- removed R14: 220k, Resistor_SMD:R_0805_2012Metric_Pad1.20x1.40mm_HandSolder
- removed R15: 30k, Resistor_SMD:R_0805_2012Metric_Pad1.20x1.40mm_HandSolder
- removed R16(PG_pull_up)101, R2: 100k, Resistor_SMD:R_0805_2012Metric_Pad1.20x1.40mm_HandSolder
- removed R27: NC, Resistor_SMD:R_0805_2012Metric_Pad1.20x1.40mm_HandSolder
- removed U4: TPS54538RQFR, RF:TPS54538RQFR
- added BU101: ~, Connector:FanPinHeader_1x03_P2.54mm_Vertical, F.Cu at (96.8, 104.4)
- added C101: 330u, Capacitor_SMD:C_0805_2012Metric_Pad1.18x1.45mm_HandSolder, F.Cu at (101.6, 113.2)
- added C102: 22u, Capacitor_SMD:C_0805_2012Metric_Pad1.18x1.45mm_HandSolder, F.Cu at (89.5, 110.4)
- added C103: 2.2u, Capacitor_SMD:C_0805_2012Metric_Pad1.18x1.45mm_HandSolder, F.Cu at (101.5, 110.4)
- added C104: 1u, Capacitor_SMD:C_0805_2012Metric_Pad1.18x1.45mm_HandSolder, F.Cu at (101.5, 104.5)
- added C27: 22pF, Capacitor_SMD:C_0603_1608Metric_Pad1.08x0.95mm_HandSolder, F.Cu at (107.5, 87.8)
- added C28: 22pF, Capacitor_SMD:C_0603_1608Metric_Pad1.08x0.95mm_HandSolder, F.Cu at (113.4, 83.4)
- added D104: D_Schottky, Diode_SMD:D_SMA, F.Cu at (85.8, 128.7)
- added H101: MountingHole, MountingHole:MountingHole_3.2mm_M3, F.Cu at (152.3, 140.4)
- added H102: MountingHole, MountingHole:MountingHole_3.2mm_M3, F.Cu at (81.1, 109.7)
- added H103: MountingHole, MountingHole:MountingHole_3.2mm_M3, F.Cu at (113.3, 72.6)
- added L101: 1mH, Inductor_SMD:L_0805_2012Metric_Pad1.05x1.20mm_HandSolder, F.Cu at (101.6, 107.8)
- added L102: 1mH, Inductor_SMD:L_0805_2012Metric_Pad1.05x1.20mm_HandSolder, F.Cu at (104.9, 109.2)
- added Y1: 8Mhz, Crystal:Crystal_SMD_5032-4Pin_5.0x3.2mm, F.Cu at (111.6, 87.6)
- D102: value TVS -> D_Schottky; footprint Diode_SMD:D_SOD-123 -> Diode_SMD:D_SMA
- J4: footprint Connector_Coaxial:BNC_Amphenol_B6252HB-NPP3G-50_Horizontal -> Connector_Coaxial:U.FL_Hirose_U.FL-R-SMT-1_Vertical
- J5: footprint Connector_PinHeader_2.54mm:PinHeader_1x02_P2.54mm_Horizontal -> Connector_Molex:Molex_Micro-Fit_3.0_43650-0200_1x02_P3.00mm_Horizontal
- moved V_BAT+101 77.2 mm to (90.9, 119.7)
- moved J4 20.9 mm to (138.4, 113.3), turned to 180 degrees
- moved D102 3.58 mm to (85.9, 124.9)
- moved C10 3.05 mm to (124.0, 78.7)
- moved C6 3.05 mm to (117.6, 88.3)
- moved C7 3.05 mm to (117.6, 85.2)
- moved C9 3.05 mm to (121.0, 78.7)
- moved C8 3.05 mm to (117.6, 82.2)
- moved J5 1.69 mm to (86.8, 145.4), turned to 90 degrees
Connections:
- C10 pad 1: 3.3V -> +3.3V
- C2 pad 1: 3.3V -> +3.3V
- C39 pad 1: 3.3V -> +3.3V
- C40 pad 1: 3.3V -> +3.3V
- C6 pad 1: 3.3V -> +3.3V
- C7 pad 1: 3.3V -> +3.3V
- C8 pad 1: 3.3V -> +3.3V
- C9 pad 1: 3.3V -> +3.3V
- D102 pad 2: USB_5V -> BUCK_5V
- FB1 pad 2: 3.3V -> unconnected-(FB1-Pad2)
- J1 pad 4: 3.3V -> +3.3V
- R29 pad 1: 3.3V -> +3.3V
- R2_up1 pad 1: 3.3V -> +3.3V
- U1 pad 1: 3.3V -> +3.3V
- U1 pad 10: unconnected-(U1-PA0-Pad10) -> HSE_IN
- U1 pad 11: unconnected-(U1-PA1-Pad11) -> HSE_OUT
- U1 pad 24: 3.3V -> +3.3V
- U1 pad 36: 3.3V -> +3.3V
- U1 pad 48: 3.3V -> +3.3V
- U9 pad 22: 3.3V -> +3.3V
- U9 pad 23: 3.3V -> +3.3V
Routing:
- net BUCK_5V: track 133.9 -> 51.6 mm, vias 8 -> 0
- net USART2_LoRa1_M1: track 4.02 -> 71.1 mm, vias 1 -> 2
- net 3.3V: track 66.8 -> 0.00 mm, vias 7 -> 0
- net SPI2_SDcard_CS: track 107.6 -> 41.6 mm, vias 3 -> 2
- net +3.3V: track 58.0 -> 116.0 mm, vias 10 -> 16
- net Net-(U4-FB): track 39.3 -> 0.00 mm, vias 2 -> 0
- net GND: track 378.5 -> 346.5 mm, vias 28 -> 40
- net Net-(C41-Pad1): track 22.2 -> 0.00 mm
- net HSE_IN: track 0.00 -> 15.1 mm, vias 0 -> 2
- net HSE_OUT: track 0.00 -> 12.6 mm, vias 0 -> 2
- net Net-(U4-EN): track 8.95 -> 0.00 mm
- net Net-(J4-In): track 8.89 -> 0.12 mm
- net Net-(U4-MODE): track 8.62 -> 0.00 mm
- net Net-(BU101-VIN): track 0.00 -> 8.10 mm
- net USB_5V: track 78.3 -> 85.7 mm
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Other:
- board size 83 x 108.3 mm -> 82.2 x 108.3 mm

Commit message: new small avionic
Connections:
- U10 pad 19: unconnected-(U10-NC-Pad19) -> (no net)
Changed lines of the file:
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@@
 			(layers "F.Cu" "F.Mask" "F.SilkS" "F.Paste")
 			(roundrect_rratio 0.15)
-			(net 40 "unconnected-(U10-NC-Pad19)")
 			(pinfunction "NC")
 			(pintype "power_in+no_connect")

Commit message: 4/25 add some debugger
Parts:
- added C26: 100n, Capacitor_SMD:C_0603_1608Metric_Pad1.08x0.95mm_HandSolder, F.Cu at (136.0, 85.2)
- added J101: Conn_01x02, Connector_PinHeader_2.54mm:PinHeader_1x02_P2.54mm_Vertical, F.Cu at (129.3, 70.2)
- added J3: Conn_01x04, Connector_PinHeader_2.54mm:PinHeader_1x04_P2.54mm_Vertical, F.Cu at (125.0, 51.5)
- added R3: 10k, Resistor_SMD:R_0805_2012Metric_Pad1.20x1.40mm_HandSolder, F.Cu at (128.3, 79.2)
- added R4: 10k, Resistor_SMD:R_0805_2012Metric_Pad1.20x1.40mm_HandSolder, F.Cu at (122.0, 101.1)
- added REST: SW_Push, Button_Switch_THT:SW_PUSH_6mm_H4.3mm, F.Cu at (135.1, 82.2)
- Q1: value TSM3481CX6 RFG -> AO3401A
- moved TP1 14.4 mm to (119.3, 52.5)
- moved GND101 8.34 mm to (115.5, 52.4)
- moved 3V3 2.14 mm to (111.4, 52.3)
- moved C102 1.81 mm to (87.7, 110.3)
- moved C101 1.71 mm to (102.3, 114.8)
- moved C103 1.71 mm to (102.3, 111.9)
- moved C104 1.71 mm to (102.3, 106.0)
- moved L101 1.71 mm to (102.3, 109.4)
- moved L102 1.71 mm to (105.7, 110.8)
Connections:
- U1 pad 20: USART2_LoRa1_M1 -> BOOT1
- U1 pad 34: unconnected-(U1-PA13-Pad34) -> SWDIO
- U1 pad 37: unconnected-(U1-PA14-Pad37) -> SWCLK
- U1 pad 39: unconnected-(U1-PB3-Pad39) -> USART2_LoRa1_M1
- U1 pad 44: unconnected-(U1-BOOT0-Pad44) -> BOOT0
- U1 pad 7: unconnected-(U1-NRST-Pad7) -> RESET
- U10 pad 19: (no net) -> unconnected-(U10-NC-Pad19)
- U9 pad 11: Net-(U9-RF_IN) -> Net-(J4-In)
- U9 pad 9: Net-(U9-VCC_RF) -> unconnected-(U9-VCC_RF-Pad9)
Routing:
- net SWDIO: track 0.00 -> 39.8 mm, vias 0 -> 3
- net SWCLK: track 0.00 -> 36.0 mm, vias 0 -> 1
- net RESET: track 0.00 -> 29.5 mm, vias 0 -> 2
- net Net-(U9-SAFEBOOT_N): track 58.6 -> 76.9 mm
- net BOOT0: track 0.00 -> 12.1 mm
- net BOOT1: track 0.00 -> 10.2 mm
- net +3.3V: track 116.0 -> 121.3 mm, vias 16 -> 18
- net GND: track 346.5 -> 350.1 mm, vias 40 -> 47
- net USART2_LoRa1_M1: track 71.1 -> 74.2 mm, vias 2 -> 4
- net Net-(U9-RF_IN): track 3.03 -> 0.00 mm
- net Net-(J4-In): track 0.12 -> 3.16 mm
- net Net-(BU101-VIN): track 8.10 -> 9.37 mm
- net USART2_LoRa1_NRST: track 60.7 -> 61.9 mm, vias 2 -> 4
- net V_BAT+: track 46.6 -> 45.8 mm
- net SPI2_SDcard_CS: track 41.6 -> 42.2 mm
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Other:
- board text added: "SWDIO"

Commit message: Groung garber
Parts:
- C101: footprint Capacitor_SMD:C_0805_2012Metric_Pad1.18x1.45mm_HandSolder -> Capacitor_SMD:smd7343
- C22, C24: footprint Capacitor_SMD:C_0805_2012Metric_Pad1.18x1.45mm_HandSolder -> Capacitor_SMD:SMD3528
- moved C101 15.3 mm to (87.5, 118.7)
- moved C24 4.64 mm to (102.6, 116.5), turned to 0 degrees
- moved C22 4.17 mm to (101.4, 120.2), turned to 0 degrees
Routing:
- net Net-(C101-Pad2): track 5.19 -> 12.0 mm, vias 0 -> 2
- net +3.3V: track 121.3 -> 127.4 mm
- net V_BAT+: track 45.8 -> 51.7 mm
- net GND: track 350.1 -> 346.1 mm, vias 47 -> 50
