File: Deployment board/Deployment board.kicad_pcb (KiCad board)
At the start: 4 copper layers, 39 x 62 mm, 32 parts, among them J1 Conn_01x04, J2 Conn_01x04, J3 Conn_01x02, J4 Conn_01x02, J5 Conn_01x02, J6 REMOVE BEFORE FLIGHT, J7 Conn_01x02, Q1 IRLR7843, Q2 IRLR7843, Q3 FDD4141, Q4 IRLR7843

Commit message: jpush
Parts:
- C1: value 77-VJ0805Y104KCAAJ -> 100n
- C3: value 667-EEH-ZS1E102UP -> 1000u
- D1, D2: value 78-SD101CWS-HE3_A-08 -> D_Schottky
- D3: value 755-SML-S13UTT68 -> MFire
- D4: value 755-SML-S13UTT68 -> BFire
- D5: value 652-SMAJ15CA -> TVS
- D6: value 755-SML-S13UTT68 -> Indicater
- D7: value 750-SS54BF-HF -> D_Schottky
- D8: value 755-SML-S13UTT68 -> Motor
- F1: value 652-SF-1206HV15M-2 -> Fuse(>15A)
- J6: value REMOVE BEFORE FLIGHT -> XT60
- R1, R2, R3: value 708-RNAN0805BKE1K00 -> 1k
- R4, R5, R7, R8: value 667-ERA-6ARB332V -> 3.3k
- R6: value 594-MCU0805PC1003FP5 -> 100k
Connections:
- J3 pad 1: V_D_BAT+ -> V_Ｄ_BAT+
- J4 pad 1: V_D_BAT+ -> V_Ｄ_BAT+
Changed lines of the file:
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@@
 	(net 17 "Net-(D7-A)")
 	(net 18 "Net-(D8-K)")
+	(net 19 "V_Ｄ_BAT+")
 	(footprint "Resistor_SMD:R_0805_2012Metric_Pad1.20x1.40mm_HandSolder"
 		(placed yes)
@@
 			)
 		)
-		(property "Value" "667-ERA-6ARB332V"
+		(property "Value" "3.3k"
 			(at 0 1.65 90)
 			(layer "F.Fab")
@@
 			(remove_unused_layers no)
 			(roundrect_rratio 0.147059)
-			(net 15 "V_D_BAT+")
+			(net 19 "V_Ｄ_BAT+")
 			(pinfunction "Pin_1")
 			(pintype "passive")
@@
 			)
 		)
-		(property "Description" "Generic connector, single row, 01x04, script generated (kicad-library-utils/schlib/autogen/connector/)"
+		(property "Description" "Generic connector, single row, 01x03, script generated (kicad-library-utils/schlib/autogen/connector/)"
 			(at 0 0 0)
 			(layer "F.Fab")
@@
 			)
 		)
-		(property "Value" "78-SD101CWS-HE3_A-08"
+		(property "Value" "D_Schottky"
 			(at 0.1 1.9 0)
 			(layer "F.Fab")
@@
 			)
 		)
-		(property "Value" "755-SML-S13UTT68"
+		(property "Value" "Indicater"
 			(at 0 1.83 0)
 			(layer "F.Fab")
@@
 			)
 		)
-		(property "Value" "750-SS54BF-HF"
+		(property "Value" "D_Schottky"
 			(at 0 3.1 90)
 			(layer "F.Fab")
@@
 			)
 		)
-		(property "Value" "755-SML-S13UTT68"
+		(property "Value" "BFire"
 			(at 0 1.83 90)
 			(layer "F.Fab")
@@
 			)
 		)
-		(property "Value" "77-VJ0805Y104KCAAJ"
+		(property "Value" "100n"
 			(at 0 1.68 90)
 			(layer "F.Fab")
@@
 			)
 		)
-		(property "Value" "667-ERA-6ARB332V"
+		(property "Value" "3.3k"
 			(at 0 1.65 90)
 			(layer "F.Fab")
@@
 			)
 		)
-		(property "Value" "652-SF-1206HV15M-2"
+		(property "Value" "Fuse(>15A)"
 			(at 0 1.83 270)
 			(layer "F.Fab")
@@
 			)
 		)
-		(property "Value" "667-ERA-6ARB332V"
+		(property "Value" "3.3k"
 			(at 0 1.65 0)
 			(layer "F.Fab")
@@
 			)
 		)
-		(property "Value" "594-MCU0805PC1003FP5"
+		(property "Value" "100k"
 			(at 0 1.65 0)
 			(layer "F.Fab")
@@
 			)
 		)
-		(property "Value" "755-SML-S13UTT68"
+		(property "Value" "Motor"
 			(at 0 1.83 90)
 			(layer "F.Fab")
@@
 			)
 		)
-		(property "Value" "708-RNAN0805BKE1K00"
+		(property "Value" "1k"
 			(at 0 1.65 90)
 			(layer "F.Fab")
@@
 			)
 		)
-		(property "Value" "667-EEH-ZS1E102UP"
+		(property "Value" "1000u"
 			(at 0 6.3 0)
 			(layer "F.Fab")
@@
 			)
 		)
-		(property "Value" "708-RNAN0805BKE1K00"
+		(property "Value" "1k"
 			(at 0 1.65 90)
 			(layer "F.Fab")
@@
 			)
 		)
-		(property "Description" "Generic connector, single row, 01x04, script generated (kicad-library-utils/schlib/autogen/connector/)"
+		(property "Description" "Generic connector, single row, 01x03, script generated (kicad-library-utils/schlib/autogen/connector/)"
 			(at 0 0 0)
 			(layer "F.Fab")
@@
 			)
 		)
-		(property "Value" "REMOVE BEFORE FLIGHT"
+		(property "Value" "XT60"
 			(at -3.6 4 0)
 			(layer "F.Fab")
@@
 			)
 		)
-		(property "Value" "78-SD101CWS-HE3_A-08"
+		(property "Value" "D_Schottky"
 			(at 0.1 1.9 0)
 			(layer "F.Fab")
@@
 			(remove_unused_layers no)
 			(roundrect_rratio 0.147059)
-			(net 15 "V_D_BAT+")
+			(net 19 "V_Ｄ_BAT+")
 			(pinfunction "Pin_1")
 			(pintype "passive")
@@
 			)
 		)
-		(property "Value" "652-SMAJ15CA"
+		(property "Value" "TVS"
 			(at 0 3.1 0)
 			(layer "F.Fab")
@@
 			)
 		)
-		(property "Value" "755-SML-S13UTT68"
+		(property "Value" "MFire"
 			(at 0 1.83 90)
 			(layer "F.Fab")
@@
 			)
 		)
-		(property "Value" "667-ERA-6ARB332V"
+		(property "Value" "3.3k"
 			(at 0 1.65 90)
 			(layer "F.Fab")
@@
 			)
 		)
-		(property "Value" "708-RNAN0805BKE1K00"
+		(property "Value" "1k"
 			(at 0 1.65 0)
 			(layer "F.Fab")
