File: Deployment board/Deployment board.kicad_sch (KiCad schematic)
At the start: 28 parts, among them J1 Conn_01x04, J2 Conn_01x04, J3 Conn_01x02, J4 Conn_01x02, J5 Conn_01x02, J6 REMOVE BEFORE FLIGHT, M1 Motor_Servo, Q1 IRLR7843, Q2 IRLR7843, Q3 To be determined

Commit message: jpush
Parts:
- J1, J2: footprint Connector_PinSocket_2.54mm:PinSocket_1x04_P2.54mm_Horizontal -> Connector_PinSocket_2.54mm:PinSocket_1x04_P2.54mm_Vertical
- J3, J4: footprint Connector_PinSocket_2.54mm:PinSocket_1x02_P2.54mm_Horizontal -> Connector_PinSocket_2.54mm:PinSocket_1x02_P2.54mm_Vertical
- M1: footprint Connector_PinHeader_2.54mm:PinHeader_1x03_P2.54mm_Horizontal -> Connector_PinHeader_2.54mm:PinHeader_1x03_P2.54mm_Vertical
Changed lines of the file:
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@@
 			)
 		)
-		(property "Footprint" "Connector_PinHeader_2.54mm:PinHeader_1x03_P2.54mm_Horizontal"
+		(property "Footprint" "Connector_PinHeader_2.54mm:PinHeader_1x03_P2.54mm_Vertical"
 			(at 74.93 49.276 0)
 			(effects
@@
 			)
 		)
-		(property "Footprint" "Connector_PinSocket_2.54mm:PinSocket_1x02_P2.54mm_Horizontal"
+		(property "Footprint" "Connector_PinSocket_2.54mm:PinSocket_1x02_P2.54mm_Vertical"
 			(at 102.87 86.36 0)
 			(effects
@@
 			)
 		)
-		(property "Footprint" "Connector_PinSocket_2.54mm:PinSocket_1x04_P2.54mm_Horizontal"
+		(property "Footprint" "Connector_PinSocket_2.54mm:PinSocket_1x04_P2.54mm_Vertical"
 			(at 71.12 144.78 0)
 			(effects
@@
 			)
 		)
-		(property "Footprint" "Connector_PinSocket_2.54mm:PinSocket_1x02_P2.54mm_Horizontal"
+		(property "Footprint" "Connector_PinSocket_2.54mm:PinSocket_1x02_P2.54mm_Vertical"
 			(at 102.87 106.68 0)
 			(effects
@@
 			)
 		)
-		(property "Footprint" "Connector_PinSocket_2.54mm:PinSocket_1x04_P2.54mm_Horizontal"
+		(property "Footprint" "Connector_PinSocket_2.54mm:PinSocket_1x04_P2.54mm_Vertical"
 			(at 25.4 144.78 0)
 			(effects

Commit message: jpush
Parts:
- J5: footprint Connector_Wire:SolderWire-2sqmm_1x02_P7.8mm_D2mm_OD3.9mm -> Connector_JST:JST_EH_B2B-EH-A_1x02_P2.50mm_Vertical
- J6: footprint Connector_Wire:SolderWire-2sqmm_1x02_P7.8mm_D2mm_OD3.9mm -> Connector_AMASS:AMASS_XT60PW-F_1x02_P7.20mm_Horizontal
Connections:
- net V_D_BAT+: now also C1.1, C2.1, M1.2 (+)
- net V_Ｄ_BAT+: no longer C1.1, C2.1, M1.2 (+)
Changed lines of the file:
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@@
 			)
 		)
-		(property "Footprint" "Connector_Wire:SolderWire-2sqmm_1x02_P7.8mm_D2mm_OD3.9mm"
+		(property "Footprint" "Connector_AMASS:AMASS_XT60PW-F_1x02_P7.20mm_Horizontal"
 			(at 176.53 30.48 0)
 			(effects
@@
 			)
 		)
-		(property "Value" "V_Ｄ_BAT+"
+		(property "Value" "V_D_BAT+"
 			(at 35.56 44.4499 90)
 			(effects
@@
 			)
 		)
-		(property "Footprint" "Connector_Wire:SolderWire-2sqmm_1x02_P7.8mm_D2mm_OD3.9mm"
+		(property "Footprint" "Connector_JST:JST_EH_B2B-EH-A_1x02_P2.50mm_Vertical"
 			(at 130.81 30.48 0)
 			(effects

Commit message: add sw
Parts:
- removed M1: Motor_Servo, Connector_PinHeader_2.54mm:PinHeader_1x03_P2.54mm_Vertical, symbol Motor:Motor_Servo
- added D7: D_Schottky, Diode_SMD:D_0805_2012Metric_Pad1.15x1.40mm_HandSolder, symbol Device:D_Schottky
- added D8: Motor, LED_SMD:LED_1206_3216Metric_Pad1.42x1.75mm_HandSolder, symbol Device:LED
- added J7: Conn_01x02, Connector_JST:JST_EH_B2B-EH-A_1x02_P2.50mm_Vertical, symbol Connector_Generic:Conn_01x02
- added Q4: NMOS, symbol Simulation_SPICE:NMOS
- added R8: 3.3k, Resistor_SMD:R_0805_2012Metric_Pad1.20x1.40mm_HandSolder, symbol Device:R
- D3: value LED -> MFire
- D4: value LED -> BFire
- D6: value B_3V3 -> Indicator
- R7: value 1k -> 3.3k
Connections:
- net GND: now also C2.1, Q4.3 (S), R8.1; no longer C1.2, C2.2
- net V_D_BAT+: now also C1.2, C2.2, D7.1 (K), J7.1 (Pin_1); no longer C1.1, C2.1
- net V_Ｄ_BAT+: now also J4.1 (Pin_1); no longer J4.2 (Pin_2)
- net at D1.1 (K), D2.1 (K), R3.1: now also Q4.2 (G)
- net at D4.2 (A), Q2.1 (D): now also J4.2 (Pin_2); no longer J4.1 (Pin_1)
- new net: D8.1 (K), R8.2
- new net: C1.1, D7.2 (A), D8.2 (A), J7.2 (Pin_2), Q4.1 (D)
Other:
- note added: "12V馬達"
- note added: "3s電源輸入"
- note added: "D1、D2形成or gate(防止電流相互倒灌) Q4(NMOS)作為開關 R3下拉電阻"
- note added: "D7防馬達斷電突波 C1防雜訊 C2防馬達啟動瞬間掉電壓"
- note added: "F1保線絲 D5防突波 R6下拉電阻 Q3(PMOS)開關(防反接保護) J6物理開關 BAT+作為整体電源+"
- note added: "跟馬達那邊一樣的開關 LED用來確認電熱絲迴路是通的"
- moved on the sheet: C1, C2, R3

Commit message: finish deployment pcb
Parts:
- removed C2: 1000u, Capacitor_THT:C_Radial_D8.0mm_H7.0mm_P3.50mm, symbol Device:C
- added C3: 667-EEH-ZS1E102UP(1000u), Capacitor_SMD:CP_Elec_10x14.3, symbol Device:C_Polarized
- D1, D2: value D_Schottky -> 78-SD101CWS-HE3_A-08; footprint Diode_SMD:D_0805_2012Metric_Pad1.15x1.40mm_HandSolder -> Diode_SMD:D_SOD-323_HandSoldering
- D3: value MFire -> LED
- D4: value BFire -> LED
- D6: value Indicator -> LED
- D7: value D_Schottky -> SS54; footprint Diode_SMD:D_0805_2012Metric_Pad1.15x1.40mm_HandSolder -> Diode_SMD:D_SMA-SMB_Universal_Handsoldering
- D8: value Motor -> LED
- J1, J2: footprint Connector_PinSocket_2.54mm:PinSocket_1x04_P2.54mm_Vertical -> Connector_JST:JST_GH_BM03B-GHS-TBT_1x03-1MP_P1.25mm_Vertical
- J3, J4: footprint Connector_PinSocket_2.54mm:PinSocket_1x02_P2.54mm_Vertical -> Connector_JST:JST_EH_B2B-EH-A_1x02_P2.50mm_Vertical
- Q3: value To be determined -> RM40P40LD; footprint Package_TO_SOT_SMD:SOT-23 -> Package_TO_SOT_SMD:TO-252-2
- Q4: value NMOS -> IRLR7843; footprint (none) -> Package_TO_SOT_SMD:TO-252-2
Connections:
- net GND: now also C3.2
- net V_D_BAT+: now also C3.1
