File: Deployment board/Deployment board.kicad_sch (KiCad schematic)
At the start: 32 parts, among them J1 Conn_01x04, J2 Conn_01x04, J3 Conn_01x02, J4 Conn_01x02, J5 Conn_01x02, J6 REMOVE BEFORE FLIGHT, J7 Conn_01x02, Q1 IRLR7843, Q2 IRLR7843, Q3 FDD4141, Q4 IRLR7843

Commit message: jpush
Parts:
- C1: value 77-VJ0805Y104KCAAJ -> 100n
- C3: value 667-EEH-ZS1E102UP -> 1000u
- D1, D2: value 78-SD101CWS-HE3_A-08 -> D_Schottky
- D3: value 755-SML-S13UTT68 -> MFire
- D4: value 755-SML-S13UTT68 -> BFire
- D5: value 652-SMAJ15CA -> TVS
- D6: value 755-SML-S13UTT68 -> Indicater
- D7: value 750-SS54BF-HF -> D_Schottky
- D8: value 755-SML-S13UTT68 -> Motor
- F1: value 652-SF-1206HV15M-2 -> Fuse(>15A)
- J1, J2: value Conn_01x04 -> Conn_01x03; symbol Connector_Generic:Conn_01x04 -> Connector_Generic:Conn_01x03
- J6: value REMOVE BEFORE FLIGHT -> XT60
- R1, R2, R3: value 708-RNAN0805BKE1K00 -> 1k
- R4, R5, R7, R8: value 667-ERA-6ARB332V -> 3.3k
- R6: value 594-MCU0805PC1003FP5 -> 100k
Connections:
- net GND: no longer J1.4 (Pin_4), J2.4 (Pin_4)
Changed lines of the file:
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@@
 	)
 	(junction
-		(at 35.56 149.86)
-		(diameter 0)
-		(color 0 0 0 0)
-	)
-	(junction
 		(at 74.93 54.61)
 		(diameter 0)
@@
 	)
 	(junction
-		(at 81.28 149.86)
-		(diameter 0)
-		(color 0 0 0 0)
-	)
-	(junction
 		(at 109.22 45.72)
 		(diameter 0)
@@
 	(wire
 		(pts
-			(xy 81.28 149.86) (xy 81.28 152.4)
+			(xy 81.28 147.32) (xy 81.28 152.4)
 		)
 		(stroke
@@
 	(wire
 		(pts
-			(xy 76.2 149.86) (xy 81.28 149.86)
-		)
-		(stroke
-			(width 0)
-			(type default)
-		)
-	)
-	(wire
-		(pts
 			(xy 97.79 86.36) (xy 97.79 88.9)
 		)
@@
 	(wire
 		(pts
-			(xy 35.56 147.32) (xy 35.56 149.86)
+			(xy 35.56 147.32) (xy 35.56 152.4)
 		)
 		(stroke
@@
 	(wire
 		(pts
-			(xy 30.48 149.86) (xy 35.56 149.86)
-		)
-		(stroke
-			(width 0)
-			(type default)
-		)
-	)
-	(wire
-		(pts
 			(xy 59.69 41.91) (xy 62.23 41.91)
 		)
@@
 	(wire
 		(pts
-			(xy 35.56 149.86) (xy 35.56 152.4)
-		)
-		(stroke
-			(width 0)
-			(type default)
-		)
-	)
-	(wire
-		(pts
 			(xy 161.29 46.99) (xy 161.29 48.26)
 		)
@@
 	(wire
 		(pts
-			(xy 81.28 147.32) (xy 81.28 149.86)
-		)
-		(stroke
-			(width 0)
-			(type default)
-		)
-	)
-	(wire
-		(pts
 			(xy 64.77 46.99) (xy 64.77 41.91)
 		)
@@
 			)
 		)
-		(property "Value" "667-ERA-6ARB332V"
+		(property "Value" "3.3k"
 			(at 83.439 54.483 0)
 			(effects
@@
 			)
 		)
-		(property "Value" "755-SML-S13UTT68"
+		(property "Value" "MFire"
 			(at 85.09 89.2174 90)
 			(effects
@@
 			)
 		)
-		(property "Value" "755-SML-S13UTT68"
+		(property "Value" "Motor"
 			(at 83.566 48.768 90)
 			(effects
@@
 			)
 		)
-		(property "Value" "REMOVE BEFORE FLIGHT"
+		(property "Value" "XT60"
 			(at 176.53 34.29 0)
 			(effects
@@
 			)
 		)
-		(property "Value" "78-SD101CWS-HE3_A-08"
+		(property "Value" "D_Schottky"
 			(at 52.07 37.846 0)
 			(effects
@@
 			)
 		)
-		(property "Value" "594-MCU0805PC1003FP5"
+		(property "Value" "100k"
 			(at 163.322 44.45 0)
 			(effects
@@
 			)
 		)
-		(property "Value" "667-EEH-ZS1E102UP"
+		(property "Value" "1000u"
 			(at 105.156 63.5 90)
 			(effects
@@
 			)
 		)
-		(property "Value" "667-ERA-6ARB332V"
+		(property "Value" "3.3k"
 			(at 75.311 119.507 90)
 			(effects
@@
 			)
 		)
-		(property "Value" "652-SF-1206HV15M-2"
+		(property "Value" "Fuse(>15A)"
 			(at 143.51 26.67 90)
 			(effects
@@
 	)
 	(symbol
-		(lib_id "Connector_Generic:Conn_01x04")
+		(lib_id "Connector_Generic:Conn_01x03")
 		(at 71.12 144.78 0)
 		(mirror y)
@@
 			)
 		)
-		(property "Value" "Conn_01x04"
+		(property "Value" "Conn_01x03"
 			(at 71.12 138.43 0)
 			(effects
@@
 			)
 		)
-		(property "Description" "Generic connector, single row, 01x04, script generated (kicad-library-utils/schlib/autogen/connector/)"
+		(property "Description" "Generic connector, single row, 01x03, script generated (kicad-library-utils/schlib/autogen/connector/)"
 			(at 71.12 144.78 0)
 			(effects
@@
 		(pin "2"
 		)
-		(pin "4"
-		)
 		(pin "3"
 		)
@@
 			)
 		)
-		(property "Value" "667-ERA-6ARB332V"
+		(property "Value" "3.3k"
 			(at 75.311 99.187 90)
 			(effects
@@
 			)
 		)
-		(property "Value" "77-VJ0805Y104KCAAJ"
+		(property "Value" "100n"
 			(at 103.632 54.864 90)
 			(effects
@@
 			)
 		)
-		(property "Value" "652-SMAJ15CA"
+		(property "Value" "TVS"
 			(at 153.67 39.3699 90)
 			(effects
@@
 			)
 		)
-		(property "Value" "708-RNAN0805BKE1K00"
+		(property "Value" "1k"
 			(at 69.596 51.562 0)
 			(effects
@@
 			)
 		)
-		(property "Value" "755-SML-S13UTT68"
+		(property "Value" "BFire"
 			(at 85.09 109.5374 90)
 			(effects
@@
 			)
 		)
-		(property "Value" "78-SD101CWS-HE3_A-08"
+		(property "Value" "D_Schottky"
 			(at 52.07 27.686 0)
 			(effects
@@
 			)
 		)
-		(property "Value" "667-ERA-6ARB332V"
+		(property "Value" "3.3k"
 			(at 180.848 76.962 90)
 			(effects
@@
 			)
 		)
-		(property "Value" "755-SML-S13UTT68"
+		(property "Value" "Indicater"
 			(at 190.5 86.36 0)
 			(effects
@@
 	)
 	(symbol
-		(lib_id "Connector_Generic:Conn_01x04")
+		(lib_id "Connector_Generic:Conn_01x03")
 		(at 25.4 144.78 0)
 		(mirror y)
@@
 			)
 		)
-		(property "Value" "Conn_01x04"
+		(property "Value" "Conn_01x03"
 			(at 25.4 138.43 0)
 			(effects
@@
 			)
 		)
-		(property "Description" "Generic connector, single row, 01x04, script generated (kicad-library-utils/schlib/autogen/connector/)"
+		(property "Description" "Generic connector, single row, 01x03, script generated (kicad-library-utils/schlib/autogen/connector/)"
 			(at 25.4 144.78 0)
 			(effects
@@
 		(pin "2"
 		)
-		(pin "4"
-		)
 		(pin "3"
 		)
@@
 			)
 		)
-		(property "Value" "708-RNAN0805BKE1K00"
+		(property "Value" "1k"
 			(at 60.706 90.932 0)
 			(effects
@@
 			)
 		)
-		(property "Value" "708-RNAN0805BKE1K00"
+		(property "Value" "1k"
 			(at 60.706 111.252 0)
 			(effects
@@
 			)
 		)
-		(property "Value" "750-SS54BF-HF"
+		(property "Value" "D_Schottky"
 			(at 101.9175 41.91 0)
 			(effects
