File: Deployment board/Deployment board.kicad_sch (KiCad schematic)
At the start: 32 parts, among them J1 Conn_01x03, J2 Conn_01x03, J3 Conn_01x02, J4 Conn_01x02, J5 Conn_01x02, J6 XT60, J7 Conn_01x02, Q1 IRLR7843, Q2 IRLR7843, Q3 FDD4141, Q4 IRLR7843

Commit message: new deployment board
Parts:
- removed C1: 100n, Capacitor_SMD:C_0805_2012Metric_Pad1.18x1.45mm_HandSolder, symbol Device:C
- removed C3: 1000u, Capacitor_SMD:CP_Elec_10x14.3, symbol Device:C_Polarized
- removed D1: D_Schottky, Diode_SMD:D_SOD-323_HandSoldering, symbol Device:D_Schottky
- removed D4: BFire, LED_SMD:LED_1206_3216Metric_Pad1.42x1.75mm_HandSolder, symbol Device:LED
- removed D7: D_Schottky, Diode_SMD:D_SMA-SMB_Universal_Handsoldering, symbol Device:D_Schottky
- removed D8: Motor, LED_SMD:LED_1206_3216Metric_Pad1.42x1.75mm_HandSolder, symbol Device:LED
- removed J3, J4, J7: Conn_01x02, Connector_JST:JST_EH_B2B-EH-A_1x02_P2.50mm_Vertical, symbol Connector_Generic:Conn_01x02
- removed J6: XT60, Connector_AMASS:AMASS_XT60PW-F_1x02_P7.20mm_Horizontal, symbol Switch:SW_SPST
- removed Q4: IRLR7843, Package_TO_SOT_SMD:TO-252-2, symbol Simulation_SPICE:NMOS
- removed R2: 1k, Resistor_SMD:R_0805_2012Metric_Pad1.20x1.40mm_HandSolder, symbol Device:R
- added 2s+1: TestPoint, TestPoint:TestPoint_THTPad_D1.5mm_Drill0.7mm, symbol Connector:TestPoint
- added C1, C2, C5, C6: 1000u, Capacitor_SMD:CP_Elec_10x14.3, symbol Device:C_Polarized
- added C3, C4: 100n, Capacitor_SMD:C_0805_2012Metric_Pad1.18x1.45mm_HandSolder, symbol Device:C
- added C7, C8: 10uF 3.979mOhm, Capacitor_SMD:C_0805_2012Metric_Pad1.18x1.45mm_HandSolder, symbol Device:C
- added C9: 47uF 2.674mOhm Qty=3, Capacitor_SMD:C_0805_2012Metric_Pad1.18x1.45mm_HandSolder, symbol Device:C
- added D1: Motor, LED_SMD:LED_1206_3216Metric_Pad1.42x1.75mm_HandSolder, symbol Device:LED
- added D10, D11, D8, D9: D_Schottky, Diode_SMD:D_SOD-323_HandSoldering, symbol Device:D_Schottky
- added D4: D_Schottky, Diode_SMD:D_SMA-SMB_Universal_Handsoldering, symbol Device:D_Schottky
- added D7: Indicater, LED_SMD:LED_1206_3216Metric_Pad1.42x1.75mm_HandSolder, symbol Device:LED
- added J1, J2, J5: Conn_01x02, Connector_JST:JST_EH_B2B-EH-A_1x02_P2.50mm_Vertical, symbol Connector_Generic:Conn_01x02
- added JP1: Drogue, Jumper:SolderJumper-3_P1.3mm_Open_Pad1.0x1.5mm_NumberLabels, symbol Jumper:SolderJumper_3_Open
- added JP2: Main, Jumper:SolderJumper-3_P1.3mm_Open_Pad1.0x1.5mm_NumberLabels, symbol Jumper:SolderJumper_3_Open
- added M1, M2: Motor_Servo, Connector_PinHeader_2.54mm:PinHeader_1x03_P2.54mm_Vertical, symbol Motor:Motor_Servo
- added R1: 100ohm, Resistor_SMD:R_0805_2012Metric_Pad1.20x1.40mm_HandSolder, symbol Device:R
- added R11, R6: 3.3k, Resistor_SMD:R_0805_2012Metric_Pad1.20x1.40mm_HandSolder, symbol Device:R
- added R12: 10k, Resistor_SMD:R_0805_2012Metric_Pad1.20x1.40mm_HandSolder, symbol Device:R
- added R13: 866k, Resistor_SMD:R_0805_2012Metric_Pad1.20x1.40mm_HandSolder, symbol Device:R
- added R14: 6.81k, Resistor_SMD:R_0805_2012Metric_Pad1.20x1.40mm_HandSolder, symbol Device:R
- added R15: 34.8k, Resistor_SMD:R_0805_2012Metric_Pad1.20x1.40mm_HandSolder, symbol Device:R
- added R7: 1k, Resistor_SMD:R_0805_2012Metric_Pad1.20x1.40mm_HandSolder, symbol Device:R
- added U1: TPSM84824MOLR, TPSM84824:MOL0024A, symbol TPSM84824:TPSM84824MOLR
- D2: footprint Diode_SMD:D_SOD-323_HandSoldering -> Diode_SMD:D_SMA-SMB_Universal_Handsoldering
- D3: value MFire -> Motor
- Q3: footprint Package_TO_SOT_SMD:TO-252-3_TabPin2 -> Package_TO_SOT_SMD:SOT-23
- R4: value 3.3k -> 100ohm
- R5: value 3.3k -> 1k
- renumbered V_D_BAT+1 to 3s+1, J5 to J3, J1 to J4, J2 to J6, R7 to R10, R1 to R2, R6 to R9
Connections:
- net V_D_BAT+ is gone; now on net 3s+: 3s+1.1, R10.2
- net Backup_AV_FIRE: now also D11.2 (A); no longer Q2.2 (G)
- net Backup_AV_PWM_Servo: now also D9.2 (A); no longer D2.2 (A)
- net GND: now also D3.1 (K), C1.2, C2.2, C5.2, C6.2, C7.2, C8.2, D1.1 (K), D7.1 (K), M1.3 (-), M2.3 (-), R7.2, U1.12 (PGND), U1.13 (PGND), U1.14 (PGND), U1.15 (PGND), U1.18 (PGND), U1.19 (PGND), U1.20 (PGND), U1.21 (PGND); no longer R4.2, R8.1
- net Main_AV_FIRE: now also D10.2 (A); no longer Q1.2 (G), R2.1
- net Main_AV_PWM_Servo: now also D8.2 (A)
- net at R8.2: now also D3.2 (A)
- net at Q1.1 (D): now also D2.2 (A), C3.1, J1.2 (Pin_2); no longer D3.2 (A)
- net at R4.1: now also Q2.2 (G), R5.1; no longer D3.1 (K)
- net 3s+: now reaches Q3.2 (S)
- net 3s+: now also D2.1 (K), R8.1, C2.1, C3.2, C4.2, C5.1, C7.1, C8.1, D4.1 (K), J1.1 (Pin_1), J2.1 (Pin_1), J5.1 (Pin_1), R6.1, U1.11 (VIN), U1.22 (VIN)
- net at R3.1: now also Q1.2 (G), R1.1; no longer D2.1 (K)
- net at D5.2 (A2), F1.2, Q3.3 (D): now also J5.2 (Pin_2)
- net at Q2.1 (D): now also C4.1, D4.2 (A), J2.2 (Pin_2)
- new net: D8.1 (K), D9.1 (K), JP1.2 (C)
- new net: U1.16 (SW), U1.17 (SW)
- new net: R12.1, R13.2, U1.2 (FB)
- new net: C9.2, R13.1, R14.1, R15.1, U1.23 (AGND), U1.3 (AGND), U1.9 (AGND)
- new net: R15.2, U1.24 (RT_CLK)
- new net: R14.2, U1.5 (TT)
- new net: D10.1 (K), D11.1 (K), JP2.2 (C)
- new net: D7.2 (A), R11.1
- new net: D1.2 (A), R6.2
- new net 2s+: 2s+1.1, C1.1, C6.1, C9.1, M1.2 (+), M2.2 (+), R11.2, R12.2, U1.1 (VOUT), U1.8 (VOUT)
- new net 2sServo1: JP1.3 (B), M1.1 (PWM), R2.1
- new net 2sServo2: JP2.3 (B), M2.1 (PWM), R7.1
- new net 3sMotor1: JP1.1 (A), R4.2
- new net 3sMotor2: JP2.1 (A), R1.2
Other:
- note added: "(for droguo parachute deployment)"
- note added: "(for main parachute deployment)"
- note added: "2sBuck"
- note added: "2sServoMotor"
- note added: "3sMotor"
- note added: "Q4(NMOS)作為開關 R3下拉電阻"
- note added: "Remove Before Flight"
- note removed: "D1、D2形成or gate(防止電流相互倒灌) Q4(NMOS)作為開關 R3下拉電阻"
- note removed: "Heat Wire(for main parachute deployment)"
- note removed: "Servo(for drogue parachute deployment)"
- note removed: "connect to hot wire"
- note removed: "跟馬達那邊一樣的開關 LED用來確認電熱絲迴路是通的"
- moved on the sheet: D6, GND1, J4, J6, R10, R2

Commit message: jpush
Connections:
- net GND: now also C9.2, R13.1, R14.1, R15.1, U1.23 (AGND), U1.3 (AGND), U1.9 (AGND)
Changed lines of the file:
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@@
 	)
 	(junction
+		(at 323.85 104.14)
+		(diameter 0)
+		(color 0 0 0 0)
+	)
+	(junction
 		(at 300.99 60.96)
 		(diameter 0)
@@
 	(wire
 		(pts
+			(xy 323.85 104.14) (xy 346.71 104.14)
+		)
+		(stroke
+			(width 0)
+			(type default)
+		)
+	)
+	(wire
+		(pts
 			(xy 346.71 41.91) (xy 346.71 44.45)
 		)
@@
 	(wire
 		(pts
-			(xy 300.99 104.14) (xy 346.71 104.14)
+			(xy 300.99 104.14) (xy 323.85 104.14)
 		)
 		(stroke
@@
 					(unit 1)
 				)
+			)
+		)
+	)
+	(symbol
+		(lib_id "power:GND")
+		(at 323.85 104.14 0)
+		(unit 1)
+		(exclude_from_sim no)
+		(in_bom yes)
+		(on_board yes)
+		(dnp no)
+		(fields_autoplaced yes)
+		(property "Reference" "#PWR028"
+			(at 323.85 110.49 0)
+			(effects
+				(font
+					(size 1.27 1.27)
+				)
+				(hide yes)
+			)
+		)
+		(property "Value" "GND"
+			(at 323.85 109.22 0)
+			(effects
+				(font
+					(size 1.27 1.27)
+				)
+			)
+		)
+		(property "Footprint" ""
+			(at 323.85 104.14 0)
+			(effects
+				(font
+					(size 1.27 1.27)
+				)
+				(hide yes)
+			)
+		)
+		(property "Datasheet" ""
+			(at 323.85 104.14 0)
+			(effects
+				(font
+					(size 1.27 1.27)
+				)
+				(hide yes)
+			)
+		)
+		(property "Description" "Power symbol creates a global label with name \"GND\" , ground"
+			(at 323.85 104.14 0)
+			(effects
+				(font
+					(size 1.27 1.27)
+				)
+				(hide yes)
+			)
+		)
+		(pin "1"
+		)
+		(instances
+			(project ""
+				(path "/0306e6d1-d01c-48b9-a21d-45e3980b499b"
+					(reference "#PWR028")
+					(unit 1)
+				)

Commit message: finish deployment board
Parts:
- added H1, H2, H3, H4: MountingHole, MountingHole:MountingHole_2.2mm_M2, symbol Mechanical:MountingHole

Commit message: deployment board
Parts:
- removed D1, D3: Motor, LED_SMD:LED_1206_3216Metric_Pad1.42x1.75mm_HandSolder, symbol Device:LED
- removed J4, J6: Conn_01x03, Connector_JST:JST_GH_BM03B-GHS-TBT_1x03-1MP_P1.25mm_Vertical, symbol Connector_Generic:Conn_01x03
- removed J5: Conn_01x02, Connector_JST:JST_EH_B2B-EH-A_1x02_P2.50mm_Vertical, symbol Connector_Generic:Conn_01x02
- removed JP1: Drogue, Jumper:SolderJumper-3_P1.3mm_Open_Pad1.0x1.5mm_NumberLabels, symbol Jumper:SolderJumper_3_Open
- removed JP2: Main, Jumper:SolderJumper-3_P1.3mm_Open_Pad1.0x1.5mm_NumberLabels, symbol Jumper:SolderJumper_3_Open
- removed R6, R8: 3.3k, Resistor_SMD:R_0805_2012Metric_Pad1.20x1.40mm_HandSolder, symbol Device:R
- added J4, J5: Conn_01x04, Connector_JST:JST_GH_BM04B-GHS-TBT_1x04-1MP_P1.25mm_Vertical, symbol Connector_Generic:Conn_01x04
- added J6, J7: Conn_01x02, Connector_JST:JST_GH_BM02B-GHS-TBT_1x02-1MP_P1.25mm_Vertical, symbol Connector_Generic:Conn_01x02
Connections:
- net 2sServo1: now also D9.1 (K), J7.2 (Pin_2)
- net 2sServo2: now also D8.1 (K), J7.1 (Pin_1)
- net 3sMotor1: now also D11.1 (K), J6.2 (Pin_2)
- net 3sMotor2: now also D10.1 (K), J6.1 (Pin_1)
- net Backup_AV_FIRE: now also J4.3 (Pin_3)
- net Backup_AV_PWM_Servo: now also J4.4 (Pin_4)
- net GND: now also J4.1 (Pin_1), J4.2 (Pin_2), J5.1 (Pin_1), J5.2 (Pin_2)
- net Main_AV_FIRE: now also J5.3 (Pin_3)
- net Main_AV_PWM_Servo: now also J5.4 (Pin_4)
Other:
- note removed: "Remove Before Flight"
