File: BigAvionic/Second_layer_MCU/_autosave-Second_layer_MCU.kicad_sch (KiCad schematic)
At the start: 86 parts, among them J1 Conn_01x02, J10 Conn_01x04, J12 Conn_01x04, J2 USB_C_Receptacle_USB2.0_16P, J3 Conn_01x04, J4 Screw_Terminal_01x02, J6 Micro_SD_Card_Det1, J9 Conn_01x04, Q5 NMOS, SW1 SW_Push, SW2 USER_Buttom, SW3 USER_Buttom, U1 STM32F405VGTx, U12 W25Q128JVS, U5 BMI088, U6 BMP390, U8 ADXL375BCCZ, Y1 8Mhz

Commit message: finish power layer(still need check)
Connections:
- net SUP_STAT: now reaches U1.16 (PC1)
- net PG_BUCK: now reaches U1.17 (PC2)
- net +USB_5V: no longer names the net of J2.A4 (VBUS), J2.A9 (VBUS), J2.B4 (VBUS), J2.B9 (VBUS), R9.2
- no-connect marks 25 -> 23
Other:
- note added: "22ohm near mcu to prevent from ringing"
- moved on the sheet: J2, R6, R7, R9
