File: BigAvionic/Second_layer_MCU/_autosave-Second_layer_MCU.kicad_sch (KiCad schematic)
At the start: 98 parts, among them J1 Conn_01x04, J10 Conn_01x04, J11 Conn_01x04, J13 Conn_01x08, J14 Conn_01x08, J2 USB_C_Receptacle_USB2.0_16P, J3 Conn_01x02, J4 Micro_SD_Card_Det1, J5 Conn_01x04, J6 Conn_01x04, J7 Screw_Terminal_01x02, J8 Conn_01x04, J9 Conn_01x08, Q2 BSS138, SW1 SW_Push, SW2 USER_Buttom, SW3 USER_Buttom, U1 STM32F405VGTx, U2 W25Q128JVS, U3 ADXL375BCCZ, U4 BMP390, U5 BMI088, Y1 8Mhz

Commit message: finish all layer
Parts:
- SW2, SW3: footprint Button_Switch_THT:SW_PUSH_1P1T_6x3.5mm_H4.3_APEM_MJTP1243 -> Button_Switch_SMD:SW_Push_1P1T-SH_NO_CK_KMR2xxG
Changed lines of the file:
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@@
 			)
 		)
-		(property "Footprint" "Button_Switch_THT:SW_PUSH_1P1T_6x3.5mm_H4.3_APEM_MJTP1243"
+		(property "Footprint" "Button_Switch_SMD:SW_Push_1P1T-SH_NO_CK_KMR2xxG"
 			(at 400.05 304.8 0)
 			(effects
@@
 			)
 		)
-		(property "Footprint" "Button_Switch_THT:SW_PUSH_1P1T_6x3.5mm_H4.3_APEM_MJTP1243"
+		(property "Footprint" "Button_Switch_SMD:SW_Push_1P1T-SH_NO_CK_KMR2xxG"
 			(at 434.34 304.8 0)
 			(effects
