File: BigAvionic/Second_layer_MCU/Second_layer_MCU.kicad_sch (KiCad schematic)
At the start: 89 parts, among them J1 Conn_01x02, J10 Conn_01x04, J12 Conn_01x04, J2 USB_C_Receptacle_USB2.0_16P, J3 Conn_01x04, J6 Micro_SD_Card_Det1, J7 Screw_Terminal_01x01, J9 Conn_01x04, Q5 NMOS, SW1 SW_Push, SW2 USER_Buttom, SW3 USER_Buttom, U1 STM32F405VGTx, U12 W25Q128JVS, U5 BMI088, U6 BMP390, U8 ADXL375BCCZ, Y1 8Mhz

Commit message: finish power layer(still need check)
Parts:
- removed J7: Screw_Terminal_01x01, TerminalBlock_Phoenix:TerminalBlock_Phoenix_PT-1,5-2-3.5-H_1x02_P3.50mm_Horizontal, symbol Connector:Screw_Terminal_01x01
- removed R10: 0 ohm, Resistor_SMD:R_0805_2012Metric_Pad1.20x1.40mm_HandSolder, symbol Device:R
- removed R5, R54: 0ohm, Resistor_SMD:R_0805_2012Metric_Pad1.20x1.40mm_HandSolder, symbol Device:R
- added J4: Screw_Terminal_01x02, TerminalBlock_Phoenix:TerminalBlock_Phoenix_PT-1,5-2-3.5-H_1x02_P3.50mm_Horizontal, symbol Connector:Screw_Terminal_01x02
- C1, C11, C2, C20, C25, C26, C27, C28, C29, C3, C30, C31, C32, C36, C37, C4, C48, C5, C50, C51, C53, C6, C7, C8, C9: footprint Capacitor_SMD:C_0805_2012Metric_Pad1.18x1.45mm_HandSolder -> Capacitor_SMD:C_0603_1608Metric_Pad1.08x0.95mm_HandSolder
- R35, R38, R40, R41, R44: value 47k -> 10k
- Y1: footprint Crystal:Crystal_HC49-U_Vertical -> Crystal:Crystal_SMD_5032-4Pin_5.0x3.2mm
Connections:
- net GND: now also J4.1 (Pin_1), J4.2 (Pin_2)
- net HSE_OUT: now also C28.1
- net SDIO_CK: no longer R39.2
- net SDIO_CMD: now also R39.2
- net USB_D+: now also J2.A6 (D+), J2.B6 (D+)
- net USB_D-: now also J2.A7 (D-), J2.B7 (D-)
Other:
- note added: "22ohm near mcu to prevent from ringing"

Commit message: checkpoint
Connections:
- net SUP_STAT: now reaches U1.16 (PC1)
- net PG_BUCK: now reaches U1.17 (PC2)
- net +USB_5V: no longer names the net of J2.A4 (VBUS), J2.A9 (VBUS), J2.B4 (VBUS), J2.B9 (VBUS), R9.2
- no-connect marks 25 -> 23
Other:
- moved on the sheet: J2, R6, R7, R9

Commit message: add lora files
Parts:
- added J5: Conn_01x08, Connector_JST:JST_GH_SM08B-GHS-TB_1x08-1MP_P1.25mm_Horizontal, symbol Connector_Generic:Conn_01x08
Connections:
- net GND: now also J5.3 (Pin_3), J5.6 (Pin_6)
- net I2C1_SCL: now also J5.4 (Pin_4)
- net I2C1_SDA: now also J5.5 (Pin_5)
- net INT_Magn: now also J5.2 (Pin_2)
- net RST_GPS: now also J5.1 (Pin_1)
- net UART6_RX: now also J5.7 (Pin_7)
- net UART6_TX: now also J5.8 (Pin_8)
Other:
- note added: "Connection to top layer"

Commit message: add new power layer
Parts:
- added J7: Conn_01x04, Connector_JST:JST_GH_SM04B-GHS-TB_1x04-1MP_P1.25mm_Horizontal, symbol Connector_Generic:Conn_01x04
- added R1: 22ohm, Resistor_SMD:R_0805_2012Metric_Pad1.20x1.40mm_HandSolder, symbol Device:R
Connections:
- net Battery_Sensing: now also J7.1 (Pin_1)
- net GND: now also J7.4 (Pin_4)
- net PG_BUCK: now also J7.3 (Pin_3)
- net SUP_STAT: now also J7.2 (Pin_2)
- net UART3_TX: now also R1.2; no longer U1.55 (PD8)
- new net: R1.1, U1.55 (PD8)
Other:
- note added: "Connection to power layer"

Commit message: MCU process
Parts:
- removed Q5: NMOS, Package_TO_SOT_SMD:SOT-23, symbol Simulation_SPICE:NMOS
- removed R27, R36, R37, R39, R42, R43: 22ohm, Resistor_SMD:R_0805_2012Metric_Pad1.20x1.40mm_HandSolder, symbol Device:R
- added C30, C31: 22u, Capacitor_SMD:C_1206_3216Metric_Pad1.33x1.80mm_HandSolder, symbol Device:C
- added J11: Conn_01x04, Connector_JST:JST_GH_SM04B-GHS-TB_1x04-1MP_P1.25mm_Horizontal, symbol Connector_Generic:Conn_01x04
- added J13, J14: Conn_01x08, Connector_JST:JST_GH_SM08B-GHS-TB_1x08-1MP_P1.25mm_Horizontal, symbol Connector_Generic:Conn_01x08
- added Q2: BSS138, Package_TO_SOT_SMD:SOT-23, symbol Transistor_FET:BSS138
- added R1: 100k, Resistor_SMD:R_0603_1608Metric_Pad0.98x0.95mm_HandSolder, symbol Device:R
- added R19, R32, R33, R6, R7, R8, R9: 22ohm, Resistor_SMD:R_0603_1608Metric_Pad0.98x0.95mm_HandSolder, symbol Device:R
- added R35: 10k, Resistor_SMD:R_0603_1608Metric_Pad0.98x0.95mm_HandSolder, symbol Device:R
- added R4, R5: 4.7k, Resistor_SMD:R_0603_1608Metric_Pad0.98x0.95mm_HandSolder, symbol Device:R
- BZ1: footprint Buzzer_Beeper:Buzzer_12x9.5RM7.6 -> Buzzer_Beeper:MagneticBuzzer_CUI_CMT-8504-100-SMT
- D4: renamed from D12; footprint LED_SMD:LED_0805_2012Metric_Pad1.15x1.40mm_HandSolder -> Diode_SMD:D_SOD-123
- J5: renamed from J10; footprint Connector_JST:JST_EH_S4B-EH_1x04_P2.50mm_Horizontal -> Connector_JST:JST_GH_SM08B-GHS-TB_1x08-1MP_P1.25mm_Horizontal
- J6: renamed from J12; footprint Connector_JST:JST_EH_B4B-EH-A_1x04_P2.50mm_Vertical -> Connector_PinHeader_2.54mm:PinHeader_1x04_P2.54mm_Vertical
- J8: renamed from J9; footprint Connector_JST:JST_EH_S4B-EH_1x04_P2.50mm_Horizontal -> Connector_JST:JST_GH_SM04B-GHS-TB_1x04-1MP_P1.25mm_Horizontal
- R10: renamed from R44; footprint Resistor_SMD:R_0805_2012Metric_Pad1.20x1.40mm_HandSolder -> Resistor_SMD:R_0603_1608Metric_Pad0.98x0.95mm_HandSolder
- R11: renamed from R40; footprint Resistor_SMD:R_0805_2012Metric_Pad1.20x1.40mm_HandSolder -> Resistor_SMD:R_0603_1608Metric_Pad0.98x0.95mm_HandSolder
- R12: renamed from R9; footprint Resistor_SMD:R_0805_2012Metric_Pad1.20x1.40mm_HandSolder -> Resistor_SMD:R_0603_1608Metric_Pad0.98x0.95mm_HandSolder
- R13: renamed from R38; footprint Resistor_SMD:R_0805_2012Metric_Pad1.20x1.40mm_HandSolder -> Resistor_SMD:R_0603_1608Metric_Pad0.98x0.95mm_HandSolder
- R14: renamed from R41; footprint Resistor_SMD:R_0805_2012Metric_Pad1.20x1.40mm_HandSolder -> Resistor_SMD:R_0603_1608Metric_Pad0.98x0.95mm_HandSolder
- R15: renamed from R35; footprint Resistor_SMD:R_0805_2012Metric_Pad1.20x1.40mm_HandSolder -> Resistor_SMD:R_0603_1608Metric_Pad0.98x0.95mm_HandSolder
- R16: renamed from R3; footprint Resistor_SMD:R_0805_2012Metric_Pad1.20x1.40mm_HandSolder -> Resistor_SMD:R_0603_1608Metric_Pad0.98x0.95mm_HandSolder
- R17: renamed from R1; footprint Resistor_SMD:R_0805_2012Metric_Pad1.20x1.40mm_HandSolder -> Resistor_SMD:R_0603_1608Metric_Pad0.98x0.95mm_HandSolder
- R18: renamed from R4; footprint Resistor_SMD:R_0805_2012Metric_Pad1.20x1.40mm_HandSolder -> Resistor_SMD:R_0603_1608Metric_Pad0.98x0.95mm_HandSolder
- R2: renamed from R6; footprint Resistor_SMD:R_0805_2012Metric_Pad1.20x1.40mm_HandSolder -> Resistor_SMD:R_0603_1608Metric_Pad0.98x0.95mm_HandSolder
- R20: renamed from R45; footprint Resistor_SMD:R_0805_2012Metric_Pad1.20x1.40mm_HandSolder -> Resistor_SMD:R_0603_1608Metric_Pad0.98x0.95mm_HandSolder
- R21: renamed from R46; footprint Resistor_SMD:R_0805_2012Metric_Pad1.20x1.40mm_HandSolder -> Resistor_SMD:R_0603_1608Metric_Pad0.98x0.95mm_HandSolder
- R22: renamed from R47; footprint Resistor_SMD:R_0805_2012Metric_Pad1.20x1.40mm_HandSolder -> Resistor_SMD:R_0603_1608Metric_Pad0.98x0.95mm_HandSolder
- R23, R34: footprint Resistor_SMD:R_0805_2012Metric_Pad1.20x1.40mm_HandSolder -> Resistor_SMD:R_0603_1608Metric_Pad0.98x0.95mm_HandSolder
- R24: renamed from R8; footprint Resistor_SMD:R_0805_2012Metric_Pad1.20x1.40mm_HandSolder -> Resistor_SMD:R_0603_1608Metric_Pad0.98x0.95mm_HandSolder
- R25: renamed from R22; footprint Resistor_SMD:R_0805_2012Metric_Pad1.20x1.40mm_HandSolder -> Resistor_SMD:R_0603_1608Metric_Pad0.98x0.95mm_HandSolder
- R26: renamed from R28; footprint Resistor_SMD:R_0805_2012Metric_Pad1.20x1.40mm_HandSolder -> Resistor_SMD:R_0603_1608Metric_Pad0.98x0.95mm_HandSolder
- R27: renamed from R48; footprint Resistor_SMD:R_0805_2012Metric_Pad1.20x1.40mm_HandSolder -> Resistor_SMD:R_0603_1608Metric_Pad0.98x0.95mm_HandSolder
- R28: renamed from R49; footprint Resistor_SMD:R_0805_2012Metric_Pad1.20x1.40mm_HandSolder -> Resistor_SMD:R_0603_1608Metric_Pad0.98x0.95mm_HandSolder
- R29: renamed from R53; footprint Resistor_SMD:R_0805_2012Metric_Pad1.20x1.40mm_HandSolder -> Resistor_SMD:R_0603_1608Metric_Pad0.98x0.95mm_HandSolder
- R3: renamed from R7; footprint Resistor_SMD:R_0805_2012Metric_Pad1.20x1.40mm_HandSolder -> Resistor_SMD:R_0603_1608Metric_Pad0.98x0.95mm_HandSolder
- R30: renamed from R50; footprint Resistor_SMD:R_0805_2012Metric_Pad1.20x1.40mm_HandSolder -> Resistor_SMD:R_0603_1608Metric_Pad0.98x0.95mm_HandSolder
- R31: renamed from R51; footprint Resistor_SMD:R_0805_2012Metric_Pad1.20x1.40mm_HandSolder -> Resistor_SMD:R_0603_1608Metric_Pad0.98x0.95mm_HandSolder
- Y1: footprint Crystal:Crystal_SMD_5032-4Pin_5.0x3.2mm -> Crystal:Crystal_SMD_3225-4Pin_3.2x2.5mm_HandSoldering
- renumbered C10 to C1, C8 to C10, C9 to C11, C47 to C12, C48 to C13, C20 to C14, C25 to C15, C11 to C16, C27 to C17, C28 to C18, C38 to C19, C3 to C2, C36 to C20, C49 to C21, C37 to C22, C29 to C23, C50 to C24, C30 to C25, C31 to C26, C32 to C27, C51 to C28, C53 to C29, C26 to C3, C2 to C8, C1 to C9, D8 to D1, D11 to D2, D5 to D3, J3 to J1, J7 to J10, J1 to J3, J6 to J4, J4 to J7, J5 to J9, U12 to U2, U8 to U3, U6 to U4
Connections:
- net V_BAT+ is gone; now on net +3.3V: BZ1.1 (+), D4.1 (K)
- net +3.3V: now also C30.1, C31.1, J11.3 (Pin_3), J11.4 (Pin_4), R35.1, R4.2, R5.1
- net Battery_Sensing: now also J10.4 (Pin_4); no longer J10.1 (Pin_1)
- net CSB_LORA920: now also J14.7 (Pin_7)
- net GND: now also J10.1 (Pin_1), J10.2 (Pin_2), C30.2, C31.2, J11.1 (Pin_1), J11.2 (Pin_2), J13.3 (Pin_3), J13.6 (Pin_6), J14.1 (Pin_1), Q2.2 (S), R1.1; no longer J10.4 (Pin_4)
- net LORA433_M0: now also J13.8 (Pin_8)
- net LORA433_M1: now also J13.7 (Pin_7)
- net LORA433_RST: now also J13.1 (Pin_1)
- net LORA920_BUSY: now also J14.8 (Pin_8)
- net LORA920_INT: now also J14.3 (Pin_3)
- net LORA920_RST: now also J14.2 (Pin_2)
- net PG_BUCK: no longer J10.3 (Pin_3)
- net RESET: now also R35.2
- net SDIO_CK: now also J4.5 (CLK), R19.2; no longer U1.80 (PC12)
- net SDIO_CMD: now also J4.3 (CMD), R11.1, R33.1; no longer U1.83 (PD2)
- net SDIO_D0: now also J4.7 (DAT0), R10.1, R6.2; no longer U1.65 (PC8)
- net SDIO_D1: now also J4.8 (DAT1), R14.1, R7.2; no longer U1.66 (PC9)
- net SDIO_D2: now also J4.1 (DAT2), R15.1, R8.2; no longer R34.2, U1.78 (PC10)
- net SDIO_D3: now also J4.2 (DAT3/CD), R13.1, R9.2; no longer U1.79 (PC11)
- net SPI3_MISO: now also J14.4 (Pin_4)
- net SPI3_MOSI: now also J14.5 (Pin_5)
- net SPI3_SCK: now also J14.6 (Pin_6)
- net SUP_STAT: now also J10.3 (Pin_3); no longer J10.2 (Pin_2)
- net UART3_RX: now also J13.4 (Pin_4)
- net UART3_TX: now also J13.5 (Pin_5)
- net UART6_RX: now also R34.2
- net UART6_TX: now also R32.2; no longer U1.63 (PC6)
- net USER_BT1: now also R4.1
- net USER_BT2: now also R5.2
- net at BZ1.2 (-), D4.2 (A): now also Q2.3 (D)
- net at R30.1, R31.1: now also Q2.1 (G)
- net at U1.64 (PC7): now also R34.1
- net at J2.A4 (VBUS), J2.A9 (VBUS), J2.B4 (VBUS)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: now also R1.2
- new net: R7.1, U1.66 (PC9)
- new net: R9.1, U1.79 (PC11)
- new net: R32.1, U1.63 (PC6)
- new net: R6.1, U1.65 (PC8)
- new net: R8.1, U1.78 (PC10)
- new net: R19.1, U1.80 (PC12)
- new net: R33.2, U1.83 (PD2)
- new net LORA433_BUSY: J13.2 (Pin_2)
Other:
- note added: "Connection to lora layer"
- moved on the sheet: C29, J10, R10, SW3

Commit message: MCU layer progress 1
Parts:
- removed R34: 22ohm, Resistor_SMD:R_0603_1608Metric_Pad0.98x0.95mm_HandSolder, symbol Device:R
- C10, C11, C13, C14, C15, C16, C2, C20, C22, C23, C24, C25, C26, C27, C28, C29, C3, C4, C5, C6, C7: footprint Capacitor_SMD:C_0603_1608Metric_Pad1.08x0.95mm_HandSolder -> Capacitor_SMD:C_0402_1005Metric_Pad0.74x0.62mm_HandSolder
- J4: footprint Connector_Card:microSD_HC_Molex_47219-2001 -> Connector_Card:microSD_HC_Molex_104031-0811
- J5: footprint Connector_JST:JST_GH_SM08B-GHS-TB_1x08-1MP_P1.25mm_Horizontal -> Connector_JST:JST_GH_SM04B-GHS-TB_1x04-1MP_P1.25mm_Horizontal
- R1, R10, R11, R12, R13, R14, R15, R16, R17, R18, R19, R2, R20, R21, R22, R23, R24, R25, R26, R27, R28, R29, R3, R30, R31, R32, R33, R35, R4, R5, R6, R7, R8, R9: footprint Resistor_SMD:R_0603_1608Metric_Pad0.98x0.95mm_HandSolder -> Resistor_SMD:R_0402_1005Metric_Pad0.72x0.64mm_HandSolder
Connections:
- net +3V3 is gone; now on net +3.3V: C1.1, C10.1, C11.1, C2.1, C4.1, C5.1, C6.1, C7.1, FB1.2, U1.100 (VDD), U1.11 (VDD), U1.19 (VDD), U1.28 (VDD), U1.50 (VDD), U1.6 (VBAT), U1.75 (VDD)
- net UART6_RX: now also U1.64 (PC7)
