File: BigAvionic/Second_layer_MCU/Second_layer_MCU.kicad_sch (KiCad schematic)
At the start: 98 parts, among them J1 Conn_01x04, J10 Conn_01x04, J11 Conn_01x04, J13 Conn_01x08, J14 Conn_01x08, J2 USB_C_Receptacle_USB2.0_16P, J3 Conn_01x02, J4 Micro_SD_Card_Det1, J5 Conn_01x04, J6 Conn_01x04, J7 Screw_Terminal_01x02, J8 Conn_01x04, J9 Conn_01x08, Q2 BSS138, SW1 SW_Push, SW2 USER_Buttom, SW3 USER_Buttom, U1 STM32F405VGTx, U2 W25Q128JVS, U3 ADXL375BCCZ, U4 BMP390, U5 BMI088, Y1 8Mhz

Commit message: version for v1 production
Parts:
- removed SW2, SW3: USER_Buttom, Button_Switch_SMD:SW_Push_1P1T-SH_NO_CK_KMR2xxG, symbol Switch:SW_Push
- added SW2, SW3: SW_Push_Shielded, Button_Switch_SMD:SW_Push_1P1T-SH_NO_CK_KMR2xxG, symbol Switch:SW_Push_Shielded
- C17, C18: value 22pF -> 10pF
- D1: value G -> Y
- D2: value R -> G
- D3: value B -> W
- Q2: value BSS138 -> AO3400A
- R27: value 2.2k -> 220
- R28, R29: value 2.2k -> 100
- U4: value BMP390 -> BMP388/390
- Y1: value 8Mhz -> FA-238 16Mhz; footprint Crystal:Crystal_SMD_3225-4Pin_3.2x2.5mm_HandSoldering -> Crystal:Crystal_SMD_SeikoEpson_FA238-4Pin_3.2x2.5mm
Connections:
- net GND: now also SW2.1, SW2.SH (B), SW3.1, SW3.SH (B)
- net USER_BT1: now also SW2.2
- net USER_BT2: now also SW3.2
Other:
- moved on the sheet: J2, R1, R12, R2, R3
