File: BigAvionic/top layer/_autosave-top_layer.kicad_pcb (KiCad board)
At the start: 4 copper layers, 68 x 68 mm, 23 parts, among them J1 Conn_01x08, J2 Conn_Coaxial, J3 Conn_01x04, U1 NEO-M9N-00B, U2 MMC5983MA

Commit message: finish power layer(still need check)
Routing:
- net GND: vias 124 -> 122
