File: BigAvionic/top layer/top_layer.kicad_sch (KiCad schematic)
At the start: 23 parts, among them J1 Conn_01x08, J2 Conn_Coaxial, J3 Conn_01x04, U1 NEO-M9N-00B, U2 MMC5983MA

Commit message: finish power layer(still need check)
Changed lines of the file:
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@@
+	)
+	(rectangle
+		(start 212.09 63.5)
+		(end 269.24 134.62)
+		(stroke
+			(width 0.1778)
+			(type dash)
+			(color 0 0 255 1)
+		)
+		(fill
+			(type none)
+		)
 	)
 	(rectangle

Commit message: finish lora & top
Parts:
- added 3V3, GND1: TestPoint, TestPoint:TestPoint_Pad_D1.0mm, symbol Connector:TestPoint
- added D2: RED_LED, LED_SMD:LED_0805_2012Metric_Pad1.15x1.40mm_HandSolder, symbol Device:LED
- added R6: 1k, Resistor_SMD:R_0805_2012Metric_Pad1.20x1.40mm_HandSolder, symbol Device:R
Connections:
- net +3.3V: now also 3V3.1, R6.2
- net GND: now also D2.1 (K), GND1.1
- new net: D2.2 (A), R6.1
Other:
- note added: "testpoint/LED"

Commit message: check lora top power generate garber
Parts:
- C4, C6, C9: footprint Capacitor_SMD:C_0805_2012Metric_Pad1.18x1.45mm_HandSolder -> Capacitor_SMD:C_1206_3216Metric_Pad1.33x1.80mm_HandSolder
Changed lines of the file:
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@@
 			)
 		)
-		(property "Footprint" "Capacitor_SMD:C_0805_2012Metric_Pad1.18x1.45mm_HandSolder"
+		(property "Footprint" "Capacitor_SMD:C_1206_3216Metric_Pad1.33x1.80mm_HandSolder"
 			(at 185.7248 114.3 0)
 			(effects
@@
 			)
 		)
-		(property "Footprint" "Capacitor_SMD:C_0805_2012Metric_Pad1.18x1.45mm_HandSolder"
+		(property "Footprint" "Capacitor_SMD:C_1206_3216Metric_Pad1.33x1.80mm_HandSolder"
 			(at 247.3452 125.73 0)
 			(effects
@@
 			)
 		)
-		(property "Footprint" "Capacitor_SMD:C_0805_2012Metric_Pad1.18x1.45mm_HandSolder"
+		(property "Footprint" "Capacitor_SMD:C_1206_3216Metric_Pad1.33x1.80mm_HandSolder"
 			(at 162.8648 72.39 0)
 			(effects

Commit message: MCU process
Connections:
- net +3.3V: now also J3.3 (Pin_3), J3.4 (Pin_4); no longer J3.1 (Pin_1), J3.2 (Pin_2)
- net GND: now also J3.1 (Pin_1), J3.2 (Pin_2); no longer J3.3 (Pin_3), J3.4 (Pin_4)
Changed lines of the file:
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@@
 	(wire
 		(pts
-			(xy 247.65 101.6) (xy 236.22 101.6)
-		)
-		(stroke
-			(width 0)
-			(type default)
-		)
-	)
-	(wire
-		(pts
 			(xy 157.48 109.22) (xy 157.48 106.68)
 		)
@@
 	(wire
 		(pts
-			(xy 156.21 114.3) (xy 166.37 114.3)
+			(xy 247.65 109.22) (xy 236.22 109.22)
 		)
 		(stroke
@@
 	(wire
 		(pts
-			(xy 198.12 114.3) (xy 198.12 115.57)
+			(xy 156.21 114.3) (xy 166.37 114.3)
 		)
 		(stroke
@@
 	(wire
 		(pts
-			(xy 186.69 106.68) (xy 198.12 106.68)
+			(xy 198.12 114.3) (xy 198.12 115.57)
 		)
 		(stroke
@@
 	(wire
 		(pts
-			(xy 154.94 59.69) (xy 163.83 59.69)
+			(xy 186.69 106.68) (xy 198.12 106.68)
 		)
 		(stroke
@@
 	(wire
 		(pts
-			(xy 167.64 57.15) (xy 167.64 77.47)
+			(xy 154.94 59.69) (xy 163.83 59.69)
 		)
 		(stroke
@@
 	(wire
 		(pts
-			(xy 64.77 33.02) (xy 78.74 33.02)
+			(xy 167.64 57.15) (xy 167.64 77.47)
 		)
 		(stroke
@@
 	(wire
 		(pts
-			(xy 247.65 106.68) (xy 236.22 106.68)
+			(xy 64.77 33.02) (xy 78.74 33.02)
 		)
 		(stroke
@@
 	(wire
 		(pts
+			(xy 247.65 101.6) (xy 236.22 101.6)
+		)
+		(stroke
+			(width 0)
+			(type default)
+		)
+	)
+	(wire
+		(pts
 			(xy 78.74 40.64) (xy 78.74 44.45)
 		)
@@
 	(wire
 		(pts
-			(xy 247.65 109.22) (xy 236.22 109.22)
+			(xy 247.65 104.14) (xy 236.22 104.14)
 		)
 		(stroke
@@
 	(wire
 		(pts
+			(xy 247.65 106.68) (xy 236.22 106.68)
+		)
+		(stroke
+			(width 0)
+			(type default)
+		)
+	)
+	(wire
+		(pts
 			(xy 154.94 52.07) (xy 177.8 52.07)
 		)
@@
 	(wire
 		(pts
-			(xy 247.65 104.14) (xy 236.22 104.14)
-		)
-		(stroke
-			(width 0)
-			(type default)
-		)
-	)
-	(wire
-		(pts
 			(xy 64.77 33.02) (xy 64.77 46.99)
 		)
@@
 	(symbol
 		(lib_id "power:+3.3V")
-		(at 236.22 101.6 90)
-		(mirror x)
+		(at 236.22 109.22 90)
 		(unit 1)
 		(exclude_from_sim no)
@@
 		(fields_autoplaced yes)
 		(property "Reference" "#PWR04"
-			(at 240.03 101.6 0)
+			(at 240.03 109.22 0)
 			(effects
 				(font
@@
 		)
 		(property "Value" "+3.3V"
-			(at 232.41 101.5999 90)
+			(at 232.41 109.2201 90)
 			(effects
 				(font
@@
 		)
 		(property "Footprint" ""
-			(at 236.22 101.6 0)
+			(at 236.22 109.22 0)
 			(effects
 				(font
@@
 		)
 		(property "Datasheet" ""
-			(at 236.22 101.6 0)
+			(at 236.22 109.22 0)
 			(effects
 				(font
@@
 		)
 		(property "Description" "Power symbol creates a global label with name \"+3.3V\""
-			(at 236.22 101.6 0)
+			(at 236.22 109.22 0)
 			(effects
 				(font
@@
 	(symbol
 		(lib_id "power:GND")
-		(at 236.22 109.22 270)
+		(at 236.22 101.6 270)
+		(mirror x)
 		(unit 1)
 		(exclude_from_sim no)
@@
 		(dnp no)
 		(property "Reference" "#PWR07"
-			(at 229.87 109.22 0)
+			(at 229.87 101.6 0)
 			(effects
 				(font
@@
 		)
 		(property "Value" "GND"
-			(at 231.14 109.22 0)
+			(at 231.14 101.6 0)
 			(effects
 				(font
@@
 		)
 		(property "Footprint" ""
-			(at 236.22 109.22 0)
+			(at 236.22 101.6 0)
 			(effects
 				(font
@@
 		)
 		(property "Datasheet" ""
-			(at 236.22 109.22 0)
+			(at 236.22 101.6 0)
 			(effects
 				(font
@@
 		)
 		(property "Description" "Power symbol creates a global label with name \"GND\" , ground"
-			(at 236.22 109.22 0)
+			(at 236.22 101.6 0)
 			(effects
 				(font
@@
 	(symbol
 		(lib_id "power:+3.3V")
-		(at 236.22 104.14 90)
-		(mirror x)
+		(at 236.22 106.68 90)
 		(unit 1)
 		(exclude_from_sim no)
@@
 		(fields_autoplaced yes)
 		(property "Reference" "#PWR05"
-			(at 240.03 104.14 0)
+			(at 240.03 106.68 0)
 			(effects
 				(font
@@
 		)
 		(property "Value" "+3.3V"
-			(at 232.41 104.1399 90)
+			(at 232.41 106.6801 90)
 			(effects
 				(font
@@
 		)
 		(property "Footprint" ""
-			(at 236.22 104.14 0)
+			(at 236.22 106.68 0)
 			(effects
 				(font
@@
 		)
 		(property "Datasheet" ""
-			(at 236.22 104.14 0)
+			(at 236.22 106.68 0)
 			(effects
 				(font
@@
 		)
 		(property "Description" "Power symbol creates a global label with name \"+3.3V\""
-			(at 236.22 104.14 0)
+			(at 236.22 106.68 0)
 			(effects
 				(font
@@
 	(symbol
 		(lib_id "power:GND")
-		(at 236.22 106.68 270)
+		(at 236.22 104.14 270)
+		(mirror x)
 		(unit 1)
 		(exclude_from_sim no)
@@
 		(dnp no)
 		(property "Reference" "#PWR06"
-			(at 229.87 106.68 0)
+			(at 229.87 104.14 0)
 			(effects
 				(font
@@
 		)
 		(property "Value" "GND"
-			(at 231.14 106.68 0)
+			(at 231.14 104.14 0)
 			(effects
 				(font
@@
 		)
 		(property "Footprint" ""
-			(at 236.22 106.68 0)
+			(at 236.22 104.14 0)
 			(effects
 				(font
@@
 		)
 		(property "Datasheet" ""
-			(at 236.22 106.68 0)
+			(at 236.22 104.14 0)
 			(effects
 				(font
@@
 		)
 		(property "Description" "Power symbol creates a global label with name \"GND\" , ground"
-			(at 236.22 106.68 0)
+			(at 236.22 104.14 0)
 			(effects
 				(font

Commit message: MCU layer progress 1
Parts:
- added D3: TVS, Diode_SMD:D_SMA, symbol Device:D_TVS_Filled
Connections:
- net +3.3V: now also D3.2 (A2)
- net GND: now also D3.1 (A1)
Changed lines of the file:
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@@
 	)
 	(junction
+		(at 226.06 118.11)
+		(diameter 0)
+		(color 0 0 0 0)
+	)
+	(junction
 		(at 74.93 46.99)
 		(diameter 0)
@@
 	(wire
 		(pts
-			(xy 234.95 118.11) (xy 240.03 118.11)
+			(xy 222.25 118.11) (xy 226.06 118.11)
 		)
 		(stroke
@@
 	(wire
 		(pts
+			(xy 226.06 118.11) (xy 240.03 118.11)
+		)
+		(stroke
+			(width 0)
+			(type default)
+		)
+	)
+	(wire
+		(pts
 			(xy 163.83 59.69) (xy 163.83 64.77)
 		)
@@
 	)
 	(symbol
+		(lib_id "Device:D_TVS_Filled")
+		(at 226.06 121.92 90)
+		(unit 1)
+		(exclude_from_sim no)
+		(in_bom yes)
+		(on_board yes)
+		(dnp no)
+		(property "Reference" "D3"
+			(at 228.6 120.6499 90)
+			(effects
+				(font
+					(size 1.27 1.27)
+				)
+				(justify right)
+			)
+		)
+		(property "Value" "TVS"
+			(at 228.6 123.1899 90)
+			(effects
+				(font
+					(size 1.27 1.27)
+				)
+				(justify right)
+			)
+		)
+		(property "Footprint" "Diode_SMD:D_SMA"
+			(at 226.06 121.92 0)
+			(effects
+				(font
+					(size 1.27 1.27)
+				)
+				(hide yes)
+			)
+		)
+		(property "Datasheet" "~"
+			(at 226.06 121.92 0)
+			(effects
+				(font
+					(size 1.27 1.27)
+				)
+				(hide yes)
+			)
+		)
+		(property "Description" "Bidirectional transient-voltage-suppression diode, filled shape"
+			(at 226.06 121.92 0)
+			(effects
+				(font
+					(size 1.27 1.27)
+				)
+				(hide yes)
+			)
+		)
+		(pin "1"
+		)
+		(pin "2"
+		)
+		(instances
+			(project "top_layer"
+				(path "/86f02ced-935e-4813-a277-f481a37622b0"
+					(reference "D3")
+					(unit 1)
+				)
+			)
+		)
+	)
+	(symbol
 		(lib_id "Mechanical:MountingHole")
 		(at 238.76 152.4 0)
@@
 	(symbol
 		(lib_id "power:+3.3V")
-		(at 234.95 118.11 90)
+		(at 222.25 118.11 90)
 		(mirror x)
 		(unit 1)
@@
 		(fields_autoplaced yes)
 		(property "Reference" "#PWR03"
-			(at 238.76 118.11 0)
+			(at 226.06 118.11 0)
 			(effects
 				(font
@@
 		)
 		(property "Value" "+3.3V"
-			(at 231.14 118.1099 90)
+			(at 218.44 118.1099 90)
 			(effects
 				(font
@@
 		)
 		(property "Footprint" ""
-			(at 234.95 118.11 0)
+			(at 222.25 118.11 0)
 			(effects
 				(font
@@
 		)
 		(property "Datasheet" ""
-			(at 234.95 118.11 0)
+			(at 222.25 118.11 0)
 			(effects
 				(font
@@
 		)
 		(property "Description" "Power symbol creates a global label with name \"+3.3V\""
-			(at 234.95 118.11 0)
+			(at 222.25 118.11 0)
 			(effects
 				(font
@@
 					(unit 1)
 				)
+			)
+		)
+	)
+	(symbol
+		(lib_id "power:GND")
+		(at 226.06 125.73 0)
+		(unit 1)
+		(exclude_from_sim no)
+		(in_bom yes)
+		(on_board yes)
+		(dnp no)
+		(property "Reference" "#PWR09"
+			(at 226.06 132.08 0)
+			(effects
+				(font
+					(size 1.27 1.27)
+				)
+				(hide yes)
+			)
+		)
+		(property "Value" "GND"
+			(at 226.06 130.81 0)
+			(effects
+				(font
+					(size 1.27 1.27)
+				)
+				(hide yes)
+			)
+		)
+		(property "Footprint" ""
+			(at 226.06 125.73 0)
+			(effects
+				(font
+					(size 1.27 1.27)
+				)
+				(hide yes)
+			)
+		)
+		(property "Datasheet" ""
+			(at 226.06 125.73 0)
+			(effects
+				(font
+					(size 1.27 1.27)
+				)
+				(hide yes)
+			)
+		)
+		(property "Description" "Power symbol creates a global label with name \"GND\" , ground"
+			(at 226.06 125.73 0)
+			(effects
+				(font
+					(size 1.27 1.27)
+				)
+				(hide yes)
+			)
+		)
+		(pin "1"
+		)
+		(instances
+			(project "top_layer"
+				(path "/86f02ced-935e-4813-a277-f481a37622b0"
+					(reference "#PWR09")
+					(unit 1)
+				)
