File: SmallAvionic/Joyce2/SmallAvionic.kicad_sch (KiCad schematic)
At the start: 103 parts, among them J1 Conn_01x02, J2 Boot_mode_pin, J3 Conn_01x04, J4 USB_C_Receptacle_USB2.0_16P, J5 Conn_01x04, J6 Conn_01x04, J7 Screw_Terminal_01x01, J8 Conn_01x03, Q1 TSM3481CX6 RFG, Q2 TSM3481CX6 RFG, Q3 NMOS, SW1 SW_Push, SW2 USER_Buttom, U1 LD1117S33TR_SOT223, U2 STM32F103C8Tx, U3 LTC4412xS6, U4 TPS54538RQFR, U5 MMC5983MA, U6 BMP390, U7 W25Q128JVS, U8 BMI088, Y1 8Mhz

Commit message: j check SmallAvionic
Connections:
- net +3.3V: now also R16(PG_pull_up)1.2
- net BUCK_5V: no longer R16(PG_pull_up)1.1
- net CSB_Flash: no longer U2.29 (PA8)
- net PG_BUCK: now also R16(PG_pull_up)1.1; no longer R16(PG_pull_up)1.2
- net RST renamed NRST
Other:
- note added: "3.3V是用於open-drain，並非電源輸出"
- note added: "C21C22負載電容， 負責與石英晶體共振"
- note added: "C26C29要記得放在VDD、VDDIO旁邊"
- note added: "C32濾波"
- note added: "C4去彈跳電容， 吸收雜訊"
- note added: "CSB上拉"
- note added: "J2拿來接跳線， 使得reset後boot0=1， 回復出廠"
- note added: "PB12 GPIO_OUT"
- note added: "SDA、SCL要上拉"
- note added: "磁珠:抑制高頻雜訊"
- note added: "類比店員"
- note removed: "3.3V是用於open-drain，並非電源輸出 R9上拉電阻，防腳位浮接"
- moved on the sheet: R16(PG_pull_up)1

Commit message: jpush
Parts:
- J5: value Conn_01x04 -> Conn_01x03; footprint (none) -> Connector_JST:JST_GH_BM03B-GHS-TBT_1x03-1MP_P1.25mm_Vertical; symbol Connector_Generic:Conn_01x04 -> Connector_Generic:Conn_01x03
Connections:
- net CSB_Flash: now also U2.29 (PA8)
- net GND: no longer J5.4 (Pin_4)
Other:
- note added: "C27在VCC旁邊 C25在3.3V旁"
Changed lines of the file:
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@@
 	)
 	(rectangle
-		(start 110.49 121.92)
-		(end 125.73 128.27)
-		(stroke
-			(width 0)
-			(type solid)
-			(color 255 0 0 1)
-		)
-		(fill
-			(type color)
-			(color 255 0 0 1)
-		)
-	)
-	(rectangle
 		(start 118.11 280.67)
 		(end 147.32 313.69)
@@
 	(rectangle
 		(start 109.22 77.47)
-		(end 121.92 99.06)
+		(end 123.19 101.6)
 		(stroke
 			(width 0)
@@
 	)
 	(rectangle
+		(start 194.31 269.24)
+		(end 209.55 274.32)
+		(stroke
+			(width 0)
+			(type solid)
+		)
+		(fill
+			(type color)
+			(color 0 255 0 1)
+		)
+	)
+	(rectangle
 		(start 241.3 260.096)
 		(end 295.91 311.15)
@@
 	)
 	(rectangle
-		(start 119.38 111.76)
-		(end 119.38 111.76)
+		(start 58.42 127)
+		(end 73.66 132.08)
 		(stroke
 			(width 0)
-			(type default)
+			(type solid)
 		)
 		(fill
-			(type none)
+			(type color)
+			(color 0 255 0 1)
 		)
 	)
 	(rectangle
-		(start 226.06 220.98)
-		(end 241.3 227.33)
+		(start 119.38 111.76)
+		(end 119.38 111.76)
 		(stroke
 			(width 0)
-			(type solid)
-			(color 255 0 0 1)
+			(type default)
 		)
 		(fill
-			(type color)
-			(color 255 0 0 1)
+			(type none)
 		)
 	)
@@
 	)
 	(rectangle
-		(start 227.33 227.33)
+		(start 227.33 224.79)
 		(end 241.3 234.95)
 		(stroke
@@
 		)
 	)
+	(text "C27在VCC旁邊\nC25在3.3V旁"
+		(exclude_from_sim no)
+		(at 310.388 250.444 0)
+		(effects
+			(font
+				(size 1.27 1.27)
+			)
+			(justify left)
+		)
+	)
 	(text "磁珠:抑制高頻雜訊"
 		(exclude_from_sim no)
@@
 	)
 	(junction
-		(at 213.36 278.13)
-		(diameter 0)
-		(color 0 0 0 0)
-	)
-	(junction
 		(at 213.36 147.32)
 		(diameter 0)
@@
 	(wire
 		(pts
-			(xy 213.36 275.59) (xy 213.36 278.13)
-		)
-		(stroke
-			(width 0)
-			(type default)
-		)
-	)
-	(wire
-		(pts
 			(xy 63.5 213.36) (xy 63.5 217.17)
 		)
@@
 	(wire
 		(pts
-			(xy 213.36 278.13) (xy 215.9 278.13)
-		)
-		(stroke
-			(width 0)
-			(type default)
-		)
-	)
-	(wire
-		(pts
 			(xy 44.45 97.79) (xy 50.8 97.79)
 		)
@@
 	(wire
 		(pts
-			(xy 215.9 275.59) (xy 213.36 275.59)
+			(xy 215.9 275.59) (xy 210.82 275.59)
 		)
 		(stroke
@@
 	(wire
 		(pts
-			(xy 210.82 278.13) (xy 213.36 278.13)
-		)
-		(stroke
-			(width 0)
-			(type default)
-		)
-	)
-	(wire
-		(pts
 			(xy 317.5 344.17) (xy 317.5 345.44)
 		)
@@
 	(wire
 		(pts
-			(xy 210.82 278.13) (xy 210.82 280.67)
+			(xy 210.82 275.59) (xy 210.82 280.67)
 		)
 		(stroke
@@
 	(global_label "CSB_Flash"
 		(shape input)
-		(at 113.03 125.73 0)
+		(at 109.22 100.33 0)
 		(fields_autoplaced yes)
 		(effects
@@
 		)
 		(property "Intersheetrefs" "${INTERSHEET_REFS}"
-			(at 125.8122 125.73 0)
+			(at 122.0022 100.33 0)
 			(effects
 				(font
@@
 	)
 	(symbol
-		(lib_id "Connector_Generic:Conn_01x04")
+		(lib_id "Connector_Generic:Conn_01x03")
 		(at 220.98 273.05 0)
 		(unit 1)
 		(exclude_from_sim no)
 		(in_bom yes)
-		(on_board yes)
+		(on_board no)
 		(dnp no)
 		(fields_autoplaced yes)
 		(property "Reference" "J5"
-			(at 223.52 273.0499 0)
+			(at 223.52 271.7799 0)
 			(effects
 				(font
@@
 			)
 		)
-		(property "Value" "Conn_01x04"
-			(at 223.52 275.5899 0)
+		(property "Value" "Conn_01x03"
+			(at 223.52 274.3199 0)
 			(effects
 				(font
@@
 			)
 		)
-		(property "Footprint" ""
+		(property "Footprint" "Connector_JST:JST_GH_BM03B-GHS-TBT_1x03-1MP_P1.25mm_Vertical"
 			(at 220.98 273.05 0)
 			(effects
@@
 			)
 		)
-		(property "Description" "Generic connector, single row, 01x04, script generated (kicad-library-utils/schlib/autogen/connector/)"
+		(property "Description" "Generic connector, single row, 01x03, script generated (kicad-library-utils/schlib/autogen/connector/)"
 			(at 220.98 273.05 0)
 			(effects
@@
 		(pin "3"
 		)
-		(pin "4"
-		)
 		(pin "2"

Commit message: jpush
Parts:
- 3V1, Buck_5v1, GND1, V_BAT+1: footprint (none) -> TestPoint:TestPoint_THTPad_D2.0mm_Drill1.0mm
- C1, C10, C11, C12, C13, C14, C15, C16, C17, C18, C19, C2, C20, C21, C22, C23, C24, C25, C26, C27, C28, C29, C3, C30, C31, C32, C33, C4, C5, C6, C7, C8, C9: footprint (none) -> Capacitor_SMD:C_0805_2012Metric_Pad1.18x1.45mm_HandSolder
- R40: renamed from 5k1; value 10k -> 5k
Connections:
- net PG_BUCK: now also U2.39 (PB3)
- net SUP_STAT: now also U2.40 (PB4)
Other:
- note added: "C30濾波"
- note added: "C33濾波"
- note added: "I2C感測器預留接口 (磁力計那邊上拉過了)"
- note added: "V=BAT(8.4)*5/(5+10)=2.8V"
- note added: "VG-VS>Vth -->open"
- note added: "讓大小航電板共地"
- note added: "防反向突波"
