File: SmallAvionic/Joyce2/SmallAvionic.kicad_pcb (KiCad board)
At the start: 4 copper layers, 58.2 x 76.6 mm, 103 parts, among them J1 Conn_01x02, J2 Boot_mode_pin, J3 Conn_01x04, J4 USB_C_Receptacle_USB2.0_16P, J5 Conn_01x03, J6 Conn_01x04, J7 Screw_Terminal_01x01, J8 Conn_01x03, Q1 TSM3481CX6 RFG, Q2 TSM3481CX6 RFG, Q3 NMOS, SW1 SW_Push, SW2 USER_Buttom, U1 LD1117S33TR_SOT223, U2 STM32F103C8Tx, U3 LTC4412xS6, U4 TPS54538RQFR, U5 MMC5983MA, U6 BMP390, U7 W25Q128JVS, U8 BMI088, Y1 8Mhz

Commit message: new small avionic
Parts:
- removed C10, C14, C7: 47u, Capacitor_SMD:C_0805_2012Metric_Pad1.18x1.45mm_HandSolder
- removed C12, C5, C9: 4.7u, Capacitor_SMD:C_0805_2012Metric_Pad1.18x1.45mm_HandSolder
- removed C15: 100n, Capacitor_SMD:C_0805_2012Metric_Pad1.18x1.45mm_HandSolder
- removed C19: 10p, Capacitor_SMD:C_0805_2012Metric_Pad1.18x1.45mm_HandSolder
- removed L1: 6.8u, Inductor_SMD:L_0805_2012Metric_Pad1.05x1.20mm_HandSolder
- removed R11, R16(PG_pull_up)1: 100k, Resistor_SMD:R_0805_2012Metric_Pad1.20x1.40mm_HandSolder
- removed R12: 390k, Resistor_SMD:R_0805_2012Metric_Pad1.20x1.40mm_HandSolder
- removed R4: 18k, Resistor_SMD:R_0805_2012Metric_Pad1.20x1.40mm_HandSolder
- removed R6: 220k, Resistor_SMD:R_0805_2012Metric_Pad1.20x1.40mm_HandSolder
- removed R8: 30k, Resistor_SMD:R_0805_2012Metric_Pad1.20x1.40mm_HandSolder
- removed U4: TPS54538RQFR, Small_av_joyce_lib:VQFN-HR9_RQF_TEX
- added BU101: ~, Connector:FanPinHeader_1x03_P2.54mm_Vertical, F.Cu at (98.0, 119.8)
- added C101: 330u, Capacitor_SMD:C_0805_2012Metric_Pad1.18x1.45mm_HandSolder, F.Cu at (105.7, 108.2)
- added C102: 22u, Capacitor_SMD:C_0805_2012Metric_Pad1.18x1.45mm_HandSolder, F.Cu at (88.6, 122.0)
- added C103: 2.2u, Capacitor_SMD:C_0805_2012Metric_Pad1.18x1.45mm_HandSolder, F.Cu at (102.2, 108.2)
- added C104: 1u, Capacitor_SMD:C_0805_2012Metric_Pad1.18x1.45mm_HandSolder, F.Cu at (102.4, 112.6)
- added J9: Conn_01x02, Connector_JST:JST_EH_B2B-EH-A_1x02_P2.50mm_Vertical, F.Cu at (116.2, 109.8)
- added L101: 1mH, Inductor_SMD:L_0805_2012Metric_Pad1.05x1.20mm_HandSolder, F.Cu at (98.2, 113.2)
- added L102: 1mH, Inductor_SMD:L_0805_2012Metric_Pad1.05x1.20mm_HandSolder, F.Cu at (105.8, 112.5)
- moved R15 228.2 mm to (17.9, 121.6)
- moved D2 225.2 mm to (18.0, 116.8)
- moved D3 219.9 mm to (21.0, 116.8)
- moved R16 218.4 mm to (20.9, 121.6)
- moved R32 205.3 mm to (36.8, 147.2)
- moved C33 202.8 mm to (36.8, 144.2)
- moved R40 201.4 mm to (36.8, 150.1)
- moved BZ1 194.0 mm to (31.9, 32.0)
- moved R28 193.6 mm to (29.8, 47.6)
- moved R29 193.5 mm to (29.8, 50.6)
- moved R25 187.0 mm to (29.8, 44.7)
- moved D6 186.9 mm to (33.7, 42.0)
- moved J6 185.3 mm to (67.1, 22.3)
- moved J4 184.7 mm to (58.7, 91.8), turned to -90 degrees
- moved D5 179.1 mm to (36.7, 46.2)
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Connections:
- U2 pad 39: PG_BUCK -> unconnected-(U2-PB3-Pad39)
Routing:
- net GND: track 319.4 -> 15.1 mm, vias 12 -> 1
- net +3.3V: track 265.5 -> 11.0 mm, vias 11 -> 0
- net V_BAT+: track 142.4 -> 0.00 mm, vias 2 -> 0
- net BUCK_5V: track 56.1 -> 0.00 mm, vias 4 -> 0
- net USART1_RX: track 54.6 -> 0.00 mm, vias 2 -> 0
- net USART1_TX: track 53.4 -> 0.00 mm, vias 2 -> 0
- net Buzzer: track 48.9 -> 0.00 mm, vias 2 -> 0
- net PG_BUCK: track 45.4 -> 0.00 mm, vias 3 -> 0
- net I2C1_SDA: track 54.6 -> 11.1 mm
- net I2C1_SCL: track 44.5 -> 7.05 mm, vias 3 -> 2
- net USB_D+: track 39.9 -> 2.50 mm, vias 2 -> 0
- net SUP_STAT: track 33.6 -> 2.37 mm, vias 2 -> 1
- net +USB_5V: track 35.7 -> 6.68 mm, vias 2 -> 1
- net USB_D-: track 29.0 -> 0.00 mm, vias 2 -> 0
- net Net-(BZ1--): track 28.6 -> 0.00 mm
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- removed copper zone on In2.Cu, net GND
Other:
- board size 58.2 x 76.6 mm -> 72.9 x 76.6 mm

Commit message: new small avionic
Parts:
- added H1: MountingHole, MountingHole:MountingHole_2.2mm_M2, F.Cu at (189.6, 111.3)
- added H2: MountingHole, MountingHole:MountingHole_2.2mm_M2, F.Cu at (254.3, 73.0)
- added H3: MountingHole, MountingHole:MountingHole_2.2mm_M2, F.Cu at (254.5, 62.5)
- added H4: MountingHole, MountingHole:MountingHole_2.2mm_M2, F.Cu at (253.2, 109.1)
- moved R29 219.9 mm to (249.1, 67.2), turned to -90 degrees
- moved BZ1 212.6 mm to (239.1, 79.5)
- moved D6 211.9 mm to (240.2, 89.8)
- moved R25 202.3 mm to (226.9, 89.9), turned to 180 degrees
- moved Q3 198.9 mm to (243.9, 64.1)
- moved C33 191.1 mm to (208.2, 59.7)
- moved R32 191.1 mm to (208.1, 62.7)
- moved R40 191.1 mm to (208.1, 65.6)
- moved D5 190.9 mm to (222.3, 90.8), turned to 180 degrees
- moved R15 183.5 mm to (200.1, 99.9), turned to 0 degrees
- moved GND1 182.2 mm to (231.2, 113.6)
- moved R16 181.1 mm to (200.3, 96.5), turned to 0 degrees
- moved D2 178.4 mm to (195.5, 99.4), turned to 180 degrees
- moved R28 176.0 mm to (204.3, 69.8), turned to -90 degrees
- moved D3 175.7 mm to (195.5, 96.3), turned to 180 degrees
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Routing:
- net +3.3V: track 11.0 -> 302.6 mm, vias 0 -> 12
- net GND: track 15.1 -> 233.0 mm, vias 1 -> 26
- net Net-(Q3-G): track 0.00 -> 53.2 mm, vias 0 -> 2
- net BUCK_5V: track 0.00 -> 48.1 mm, vias 0 -> 1
- net V_BAT+: track 0.00 -> 43.7 mm, vias 0 -> 1
- net +USB_5V: track 6.68 -> 46.1 mm, vias 1 -> 3
- net PWM Servo: track 5.52 -> 43.6 mm, vias 1 -> 2
- net FIRE: track 7.01 -> 44.0 mm, vias 1 -> 2
- net I2C1_SCL: track 7.05 -> 41.9 mm
- net I2C1_SDA: track 11.1 -> 42.6 mm
- net SWCLK: track 1.59 -> 28.8 mm
- net SWDIO: track 0.00 -> 26.3 mm, vias 0 -> 1
- net SPI2_SCK: track 0.00 -> 23.6 mm, vias 0 -> 2
- net Net-(BZ1--): track 0.00 -> 23.2 mm
- net SPI2_MOSI: track 0.00 -> 22.0 mm, vias 0 -> 2
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- added copper zone on In1.Cu, net +3.3V
- added copper zone on In1.Cu, net BUCK_5V
- added copper zone on In2.Cu, net GND
- added copper zone on In1.Cu, net V_BAT+
Other:
- board size 72.9 x 76.6 mm -> 76.8 x 61.5 mm

Commit message: smallavionic
Parts:
- C101: footprint Capacitor_SMD:C_0805_2012Metric_Pad1.18x1.45mm_HandSolder -> Capacitor_THT:CP_Radial_D6.3mm_P2.50mm
- moved R3 3.82 mm to (242.8, 94.2), turned to 90 degrees
- moved J9 3.48 mm to (248.2, 95.7)
- moved C101 2.59 mm to (236.8, 93.3)
- moved Q1 2.16 mm to (240.8, 99.3)
- moved F1 1.78 mm to (245.7, 106.6)
- moved J1 1.67 mm to (236.6, 106.0)
- moved D1 1.67 mm to (248.2, 102.3)
- moved L102 1.36 mm to (235.0, 99.0), turned to 180 degrees
Routing:
- net V_BAT+: track 43.7 -> 52.2 mm
- net +3.3V: track 302.6 -> 310.3 mm
- net Net-(C101-Pad2): track 5.57 -> 10.1 mm
- net Net-(Q3-G): track 53.2 -> 50.6 mm
- net BUCK_5V: track 48.1 -> 50.4 mm
- net unconnected-(U2-PB3-Pad39): track 1.82 -> 0.00 mm, vias 1 -> 0
- net BOOT0: track 24.3 -> 23.5 mm
- net Net-(Q1-G): track 2.88 -> 3.68 mm
- net Net-(D2-A): track 5.27 -> 4.62 mm
