File: BigAvionic/power layer/power layer.kicad_sch (KiCad schematic)
At the start: 53 parts, among them J1 Conn_01x04, J2 Conn_01x04, J3 Conn_01x04, J4 Conn_01x04, J5 Conn_01x02, Q1 TSM3481CX6 RFG, Q2 TSM3481CX6 RFG, U2 LD1117S33TR_SOT223, U3 LTC4412xS6, U4 TPS54538RQFR

Commit message: checkpoint
Parts:
- removed R16(PG_pull_up)1: 100k, Resistor_SMD:R_0805_2012Metric_Pad1.20x1.40mm_HandSolder, symbol Device:R
- added J6: USB_C_Receptacle_USB2.0_16P, Connector_USB:USB_C_Receptacle_HRO_TYPE-C-31-M-12, symbol Connector:USB_C_Receptacle_USB2.0_16P
- added R3: 100k, Capacitor_SMD:C_0603_1608Metric_Pad1.08x0.95mm_HandSolder, symbol Device:R
- added R6, R7: 5.1k, Resistor_SMD:R_0805_2012Metric_Pad1.20x1.40mm_HandSolder, symbol Device:R
- C12: footprint Capacitor_SMD:C_0805_2012Metric_Pad1.18x1.45mm_HandSolder -> Capacitor_SMD:C_0603_1608Metric_Pad1.08x0.95mm_HandSolder
- C13, C14, C15, C17, C18, C19, C22, C24: footprint Capacitor_SMD:C_0805_2012Metric_Pad1.18x1.45mm_HandSolder -> Capacitor_SMD:C_1206_3216Metric_Pad1.33x1.80mm_HandSolder
- C16: footprint Capacitor_SMD:C_0805_2012Metric_Pad1.18x1.45mm_HandSolder -> Capacitor_SMD:C_0402_1005Metric_Pad0.74x0.62mm_HandSolder
- R1, R13, R14, R15, R16, R17, R18, R19, R2, R20, R21, R52, R55: footprint Resistor_SMD:R_0805_2012Metric_Pad1.20x1.40mm_HandSolder -> Capacitor_SMD:C_0603_1608Metric_Pad1.08x0.95mm_HandSolder
- renumbered 5V to 5V1
Connections:
- net +3.3V: now also R3.1
- net +USB_5V: now also J6.A4 (VBUS), J6.A9 (VBUS), J6.B4 (VBUS), J6.B9 (VBUS)
- net GND: now also J6.A1 (GND), J6.A12 (GND), J6.B1 (GND), J6.B12 (GND), J6.S1 (SHIELD), R6.2, R7.2
- net PG_BUCK: now also R3.2
- new net: J6.A5 (CC1), R6.1
- new net: J6.B5 (CC2), R7.1
- no-connect marks 1 -> 7
Other:
- note added: "USB"
- note added: "when steady read high (3V) (open drain)"
- note removed: "when steady read high (5V)"
- moved on the sheet: H1, H2, H3, H4, J1
