File: BigAvionic/power layer_new/power layer.kicad_pcb (KiCad board)
At the start: 4 copper layers, 68 x 68 mm, 56 parts, among them J1 Conn_01x04, J2 Conn_01x04, J3 Conn_01x04, J4 Conn_01x04, J5 Conn_01x02, J6 USB_C_Receptacle_USB2.0_16P, Q1 TSM3481CX6 RFG, Q2 TSM3481CX6 RFG, U2 LD1117S33TR_SOT223, U3 LTC4412xS6, U4 TPS54538RQFR

Commit message: power layer finished
Parts:
- removed 3V3: TestPoint, TestPoint:TestPoint_Pad_D1.0mm
- removed C16: 10p, Capacitor_SMD:C_0402_1005Metric_Pad0.74x0.62mm_HandSolder
- removed C17, C18, C19, C22, C24: 47u, Capacitor_SMD:C_1206_3216Metric_Pad1.33x1.80mm_HandSolder
- removed C21, C23, C52: 100n, Capacitor_SMD:C_0805_2012Metric_Pad1.18x1.45mm_HandSolder
- removed F1: Fuse, Fuse:Fuse_0805_2012Metric_Pad1.15x1.40mm_HandSolder
- removed R13: 18k, Capacitor_SMD:C_0603_1608Metric_Pad1.08x0.95mm_HandSolder
- removed R14: 220k, Capacitor_SMD:C_0603_1608Metric_Pad1.08x0.95mm_HandSolder
- removed R15: 30k, Capacitor_SMD:C_0603_1608Metric_Pad1.08x0.95mm_HandSolder
- removed R16, R17: 1k, Capacitor_SMD:C_0603_1608Metric_Pad1.08x0.95mm_HandSolder
- removed R18, R19, R21: 100k, Capacitor_SMD:C_0603_1608Metric_Pad1.08x0.95mm_HandSolder
- removed R20: 1M, Capacitor_SMD:C_0603_1608Metric_Pad1.08x0.95mm_HandSolder
- removed R52: 10k, Capacitor_SMD:C_0603_1608Metric_Pad1.08x0.95mm_HandSolder
- removed R55: 5k, Capacitor_SMD:C_0603_1608Metric_Pad1.08x0.95mm_HandSolder
- removed U3: LTC4412xS6, Package_TO_SOT_SMD:TSOT-23-6
- removed U4: TPS54538RQFR, Tony:VQFN-HR9_RQF_TEX(TPS54538)
- added 3V3_1: TestPoint, TestPoint:TestPoint_Pad_D1.0mm, F.Cu at (204.2, 101.5)
- added 3V3_LORA1: TestPoint, TestPoint:TestPoint_Pad_D1.0mm, F.Cu at (179.9, 116.6)
- added BU1: R-78K5.0-2.0L, Tony:CONV_R-78K5.0-2.0L, F.Cu at (173.1, 80.1)
- added BU2: R-78K3.3-2.0L, Tony:CONV_R-78K5.0-2.0L, F.Cu at (202.1, 108.9)
- added C10: 100n, Capacitor_SMD:C_0805_2012Metric_Pad1.18x1.45mm_HandSolder, F.Cu at (187.7, 88.0)
- added C11: 22u, Capacitor_SMD:C_1210_3225Metric_Pad1.33x2.70mm_HandSolder, F.Cu at (182.9, 90.1)
- added C2: 22u, Capacitor_SMD:C_1210_3225Metric_Pad1.33x2.70mm_HandSolder, F.Cu at (176.6, 100.5)
- added C3: 22u, Capacitor_SMD:C_1210_3225Metric_Pad1.33x2.70mm_HandSolder, F.Cu at (181.1, 107.5)
- added C4: 100n, Capacitor_SMD:C_0805_2012Metric_Pad1.18x1.45mm_HandSolder, F.Cu at (200.7, 73.8)
- added C5: 22u, Capacitor_SMD:C_1210_3225Metric_Pad1.33x2.70mm_HandSolder, F.Cu at (172.2, 94.1)
- added C6: 22u, Capacitor_SMD:C_1210_3225Metric_Pad1.33x2.70mm_HandSolder, F.Cu at (184.8, 107.5)
- added C7: 100n, Capacitor_SMD:C_0805_2012Metric_Pad1.18x1.45mm_HandSolder, F.Cu at (200.9, 86.0)
- added C8: 47u, Capacitor_SMD:C_1210_3225Metric_Pad1.33x2.70mm_HandSolder, F.Cu at (200.7, 89.2)
- added C9: 47u, Capacitor_SMD:C_1210_3225Metric_Pad1.33x2.70mm_HandSolder, F.Cu at (200.7, 94.2)
- added C_Damping1: 22u, Capacitor_Tantalum_SMD:CP_EIA-3528-21_Kemet-B_HandSolder, F.Cu at (188.6, 107.6)
- added C_Damping2: 22u, Capacitor_Tantalum_SMD:CP_EIA-3528-21_Kemet-B_HandSolder, F.Cu at (177.7, 96.9)
- added D4: G_3V3, LED_SMD:LED_0805_2012Metric_Pad1.15x1.40mm_HandSolder, F.Cu at (196.5, 98.1)
- added L2: 4.7uH, Inductor_SMD:L_APV_ANR4020, F.Cu at (185.5, 101.4)
- added R11: 470, Resistor_SMD:R_0805_2012Metric_Pad1.20x1.40mm_HandSolder, F.Cu at (182.6, 117.6)
- added R4: 470k, Resistor_SMD:R_0805_2012Metric_Pad1.20x1.40mm_HandSolder, F.Cu at (188.6, 78.4)
- added R5: 1k, Resistor_SMD:R_0805_2012Metric_Pad1.20x1.40mm_HandSolder, F.Cu at (188.6, 63.5)
- added R6: 470, Resistor_SMD:R_0805_2012Metric_Pad1.20x1.40mm_HandSolder, F.Cu at (201.2, 98.1)
- added R7: 10k, Resistor_SMD:R_0805_2012Metric_Pad1.20x1.40mm_HandSolder, F.Cu at (164.0, 99.4)
- added R8: 5k, Resistor_SMD:R_0805_2012Metric_Pad1.20x1.40mm_HandSolder, F.Cu at (163.1, 92.2)
- added U1: LD1117S33TR_SOT223, Package_TO_SOT_SMD:SOT-223-3_TabPin2, F.Cu at (201.9, 80.0)
- 5V1, GND1: footprint TestPoint:TestPoint_Pad_1.0x1.0mm -> TestPoint:TestPoint_Pad_D1.0mm
- C1: footprint Capacitor_SMD:C_0805_2012Metric_Pad1.18x1.45mm_HandSolder -> Capacitor_SMD:C_1210_3225Metric_Pad1.33x2.70mm_HandSolder
- C12: value 100n -> 22u; footprint Capacitor_SMD:C_0603_1608Metric_Pad1.08x0.95mm_HandSolder -> Capacitor_SMD:C_1210_3225Metric_Pad1.33x2.70mm_HandSolder
- C13: value 4.7u -> 47u; footprint Capacitor_SMD:C_1206_3216Metric_Pad1.33x1.80mm_HandSolder -> Capacitor_SMD:C_1210_3225Metric_Pad1.33x2.70mm_HandSolder
- C14, C15: value 4.7u -> 100n; footprint Capacitor_SMD:C_1206_3216Metric_Pad1.33x1.80mm_HandSolder -> Capacitor_SMD:C_0805_2012Metric_Pad1.18x1.45mm_HandSolder
- D1: value G_5V -> TVS; footprint LED_SMD:LED_0805_2012Metric_Pad1.15x1.40mm_HandSolder -> Diode_SMD:D_SMA
- D2: value B_3V3 -> SS24; footprint LED_SMD:LED_0805_2012Metric_Pad1.15x1.40mm_HandSolder -> Diode_SMD:D_SMA
- D3: value TVS -> G_5V
- D5: value SS24 -> G_3V3; footprint Diode_SMD:D_SMA -> LED_SMD:LED_0805_2012Metric_Pad1.15x1.40mm_HandSolder
- L1: value 6.8u -> 4.7uH; footprint Inductor_SMD:L_7.3x7.3_H3.5 -> Inductor_SMD:L_APV_ANR4020
- Q1, Q2: value TSM3481CX6 RFG -> AO3401A
- R1: value 390k -> 100k; footprint Capacitor_SMD:C_0603_1608Metric_Pad1.08x0.95mm_HandSolder -> Resistor_SMD:R_0805_2012Metric_Pad1.20x1.40mm_HandSolder
- R2: footprint Capacitor_SMD:C_0603_1608Metric_Pad1.08x0.95mm_HandSolder -> Resistor_SMD:R_0805_2012Metric_Pad1.20x1.40mm_HandSolder
- R3: value 100k -> 1M; footprint Capacitor_SMD:C_0603_1608Metric_Pad1.08x0.95mm_HandSolder -> Resistor_SMD:R_0805_2012Metric_Pad1.20x1.40mm_HandSolder
- U2: value LD1117S33TR_SOT223 -> LTC4412xS6; footprint Package_TO_SOT_SMD:SOT-223-3_TabPin2 -> Package_TO_SOT_SMD:TSOT-23-6
- moved GND1 66.9 mm to (157.3, 109.1)
- moved D5 52.8 mm to (182.6, 121.1), turned to 180 degrees
- moved D3 48.4 mm to (193.4, 63.5)
- moved 5V1 35.3 mm to (190.5, 92.9)
- moved D2 30.7 mm to (178.4, 67.8), turned to 180 degrees
- moved C13 30.0 mm to (191.7, 69.4), turned to 90 degrees
- moved C12 29.3 mm to (186.6, 118.0), turned to -90 degrees
- moved D1 26.6 mm to (173.7, 109.3)
- moved R1 19.2 mm to (175.3, 104.7), turned to -90 degrees
- moved C15 18.3 mm to (188.2, 112.3), turned to 180 degrees
- moved R2 17.3 mm to (191.1, 82.8), turned to 90 degrees
- moved L1 15.3 mm to (170.6, 98.9), turned to 90 degrees
- moved R3 15.2 mm to (191.1, 87.2)
- moved U2 13.7 mm to (187.7, 84.2), turned to 90 degrees
- moved C14 11.9 mm to (163.0, 94.7), turned to 180 degrees
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- renumbered J5 to J1, J6 to J2, J1 to J3, J3 to J4, J4 to J5, J2 to J6, R7 to R10, R6 to R9
Connections:
- C12 pad 1: V_BAT+ -> +3.3V_LoRa
- C13 pad 1: V_BAT+ -> GND
- C13 pad 2: GND -> 5V
- C14 pad 1: V_BAT+ -> Battery_Sensing
- C15 pad 1: V_BAT+ -> +3.3V_LoRa
- D1 pad 2: Net-(D1-A) -> Net-(D1-A2)
- D2 pad 1: GND -> 5V
- D2 pad 2: Net-(D2-A) -> +USB_5V
- D3 pad 2: Net-(D3-A2) -> Net-(D3-A)
- D5 pad 1: 5V -> GND
- D5 pad 2: +USB_5V -> Net-(D5-A)
- J1 pad 1: Net-(J5-Pin_1) -> Net-(D1-A2)
- J3 pad 3: PG_BUCK -> GND
- J6 pad 1: +3.3V -> +3.3V_LoRa
- J6 pad 2: +3.3V -> +3.3V_LoRa
- L1 pad 1: BUCK_5V -> V_BAT+
- Q1 pad 3: Net-(D3-A2) -> Net-(D1-A2)
- Q2 pad 2: BUCK_5V -> 5V
- Q2 pad 3: 5V -> BUCK_5V
- R1 pad 1: Net-(U4-EN) -> Net-(Q1-G)
- R1 pad 2: V_BAT+ -> GND
- R2 pad 1: GND -> Net-(U2-CTL)
- R2 pad 2: Net-(U4-EN) -> +USB_5V
- R3 pad 1: +3.3V -> Net-(U2-CTL)
- R3 pad 2: PG_BUCK -> GND
- U2 pad 1: GND -> BUCK_5V
- U2 pad 2: +3.3V -> GND
- U2 pad 3: 5V -> Net-(U2-CTL)
Routing:
- net GND: track 208.0 -> 73.7 mm, vias 60 -> 339
- net 5V: track 26.0 -> 120.2 mm, vias 16 -> 4
- net +3.3V: track 43.0 -> 128.3 mm, vias 2 -> 10
- net PG_BUCK: track 29.7 -> 0.00 mm
- net +3.3V_LoRa: track 0.00 -> 23.2 mm
- net V_BAT+: track 42.3 -> 21.8 mm, vias 2 -> 0
- net Battery_Sensing: track 35.1 -> 16.4 mm, vias 2 -> 0
- net Net-(BU2-VIN): track 0.00 -> 12.0 mm
- net Net-(BU1-VIN): track 2.69 -> 13.1 mm
- net Net-(D1-A2): track 0.00 -> 10.4 mm
- net Net-(U2-CTL): track 0.00 -> 9.55 mm
- net +USB_5V: track 43.7 -> 35.4 mm
- net Net-(U3-CTL): track 6.88 -> 0.00 mm
- net Net-(D3-A2): track 6.04 -> 0.00 mm
- net Net-(U4-MODE): track 5.68 -> 0.00 mm
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- added copper zone on In2.Cu, net +3.3V
- removed copper zone on F.Cu, net +3.3V
- removed copper zone on F.Cu, net 5V
- removed copper zone on F.Cu, net BUCK_5V
Other:
- board text added: "Power Layer v1"

Commit message: MCU process
Other:
- board text added: "BAT"
- board text added: "P_LORA"
- board text added: "P_MCU"
- board text added: "P_TOP"
- board text added: "S_MCU"
Changed lines of the file:
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@@
 		(layer "Edge.Cuts")
+	)
+	(gr_text "P_TOP"
+		(at 210.2 93.2 0)
+		(layer "F.SilkS")
+		(effects
+			(font
+				(size 1.5 1.5)
+				(thickness 0.3)
+				(bold yes)
+			)
+			(justify left bottom)
+		)
+	)
+	(gr_text "BAT"
+		(at 165.18 121.11 0)
+		(layer "F.SilkS")
+		(effects
+			(font
+				(size 1.5 1.5)
+				(thickness 0.3)
+				(bold yes)
+			)
+			(justify left bottom)
+		)
 	)
 	(gr_text "Power Layer v1"
@@
 		(layer "F.SilkS")
 		(effects
+			(font
+				(size 1.5 1.5)
+				(thickness 0.3)
+				(bold yes)
+			)
+			(justify left bottom)
+		)
+	)
+	(gr_text "S_MCU"
+		(at 151.4 96.39 0)
+		(layer "F.SilkS")
+		(effects
+			(font
+				(size 1.5 1.5)
+				(thickness 0.3)
+				(bold yes)
+			)
+			(justify left bottom)
+		)
+	)
+	(gr_text "P_MCU"
+		(at 209.23 72.65 0)
+		(layer "F.SilkS")
+		(effects
+			(font
+				(size 1.5 1.5)
+				(thickness 0.3)
+				(bold yes)
+			)
+			(justify left bottom)
+		)
+	)
+	(gr_text "P_LORA"
+		(at 200.34 120.95 0)
+		(layer "F.SilkS")
+		(effects
