File: BigAvionic/power layer_new/power layer.kicad_pcb (KiCad board)
At the start: 4 copper layers, 68 x 68 mm, 57 parts, among them J1 Conn_01x02, J2 USB_C_Receptacle_USB2.0_16P, J3 Conn_01x04, J4 Conn_01x04, J5 Conn_01x04, J6 Conn_01x04, Q1 AO3401A, Q2 AO3401A, U1 LD1117S33TR_SOT223, U2 LTC4412xS6

Commit message: version for v1 production
Parts:
- added G***: LOGO, Lib:LOGO-10*12.1, F.Cu at (154.7, 68.5)
- R11, R6: value 470 -> 100
- R5: value 1k -> 330
Routing:
- net GND: vias 339 -> 340
Other:
- board text added: "3V3"
- board text added: "3V3_L"
- board text added: "5V"
- board text added: "BUCK_5V"
- board text added: "GND"
- board text added: "NCKU Ius Bubulae Avionics v1.0 Tony"
- board text added: "Power Layer"
- board text added: "S_POWER"
- board text added: "V_BAT+"
- board text removed: "Power Layer v1"
- board text removed: "S_MCU"
