File: BigAvionic/power layer_previous/power layer.kicad_pcb (KiCad board)
At the start: 4 copper layers, 68 x 68 mm, 56 parts, among them J1 Conn_01x04, J2 Conn_01x04, J3 Conn_01x04, J4 Conn_01x04, J5 Conn_01x02, J6 USB_C_Receptacle_USB2.0_16P, Q1 TSM3481CX6 RFG, Q2 TSM3481CX6 RFG, U2 LD1117S33TR_SOT223, U3 LTC4412xS6, U4 TPS54538RQFR

Commit message: version for v1 production
Routing:
- net GND: track 208.0 -> 210.7 mm, vias 60 -> 63
