File: BigAvionic/lora/lora.kicad_sch (KiCad schematic)
At the start: 23 parts, among them J1 Conn_01x04, J2 Conn_01x08, J3 Conn_01x08, U1 E22-400T30S, U2 E80-900M23313S

Commit message: MCU layer progress 1
Parts:
- added D2: TVS, Diode_SMD:D_SMA, symbol Device:D_TVS_Filled
Connections:
- net +3.3V: now also D2.2 (A2)
- net GND: now also D2.1 (A1)
Other:
- moved on the sheet: C7
Changed lines of the file:
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@@
 	)
 	(junction
+		(at 77.47 138.43)
+		(diameter 0)
+		(color 0 0 0 0)
+	)
+	(junction
 		(at 204.47 105.41)
 		(diameter 0)
@@
 	)
 	(junction
-		(at 200.66 68.58)
+		(at 73.66 146.05)
 		(diameter 0)
 		(color 0 0 0 0)
 	)
 	(junction
-		(at 147.32 90.17)
+		(at 200.66 68.58)
 		(diameter 0)
 		(color 0 0 0 0)
 	)
 	(junction
-		(at 78.74 138.43)
+		(at 147.32 90.17)
 		(diameter 0)
 		(color 0 0 0 0)
@@
 	)
 	(junction
+		(at 73.66 138.43)
+		(diameter 0)
+		(color 0 0 0 0)
+	)
+	(junction
 		(at 209.55 105.41)
 		(diameter 0)
@@
 	(wire
 		(pts
-			(xy 77.47 146.05) (xy 78.74 146.05)
+			(xy 69.85 146.05) (xy 73.66 146.05)
 		)
 		(stroke
@@
 	(wire
 		(pts
+			(xy 77.47 138.43) (xy 80.01 138.43)
+		)
+		(stroke
+			(width 0)
+			(type default)
+		)
+	)
+	(wire
+		(pts
 			(xy 99.06 101.6) (xy 99.06 104.14)
 		)
@@
 	(wire
 		(pts
-			(xy 78.74 138.43) (xy 68.58 138.43)
+			(xy 73.66 138.43) (xy 77.47 138.43)
 		)
 		(stroke
@@
 	(wire
 		(pts
-			(xy 80.01 138.43) (xy 78.74 138.43)
+			(xy 73.66 146.05) (xy 77.47 146.05)
 		)
 		(stroke
@@
 	(wire
 		(pts
+			(xy 73.66 138.43) (xy 68.58 138.43)
+		)
+		(stroke
+			(width 0)
+			(type default)
+		)
+	)
+	(wire
+		(pts
 			(xy 147.32 80.01) (xy 147.32 82.55)
 		)
@@
 	(symbol
 		(lib_id "Device:C")
-		(at 78.74 142.24 180)
+		(at 73.66 142.24 180)
 		(unit 1)
 		(exclude_from_sim no)
@@
 		(dnp no)
 		(property "Reference" "C7"
-			(at 74.93 143.764 0)
+			(at 69.85 143.764 0)
 			(effects
 				(font
@@
 		)
 		(property "Value" "470u"
-			(at 74.93 140.9701 0)
+			(at 69.85 140.9701 0)
 			(effects
 				(font
@@
 		)
 		(property "Footprint" "Capacitor_Tantalum_SMD:CP_EIA-7343-43_Kemet-X_HandSolder"
-			(at 77.7748 138.43 0)
+			(at 72.6948 138.43 0)
 			(effects
 				(font
@@
 		)
 		(property "Datasheet" "~"
-			(at 78.74 142.24 0)
+			(at 73.66 142.24 0)
 			(effects
 				(font
@@
 		)
 		(property "Description" "Unpolarized capacitor"
-			(at 78.74 142.24 0)
+			(at 73.66 142.24 0)
 			(effects
 				(font
@@
 	(symbol
 		(lib_id "power:GND")
-		(at 77.47 146.05 270)
+		(at 69.85 146.05 270)
 		(mirror x)
 		(unit 1)
@@
 		(dnp no)
 		(property "Reference" "#PWR022"
-			(at 71.12 146.05 0)
+			(at 63.5 146.05 0)
 			(effects
 				(font
@@
 		)
 		(property "Value" "GND"
-			(at 72.39 146.05 0)
+			(at 64.77 146.05 0)
 			(effects
 				(font
@@
 		)
 		(property "Footprint" ""
-			(at 77.47 146.05 0)
+			(at 69.85 146.05 0)
 			(effects
 				(font
@@
 		)
 		(property "Datasheet" ""
-			(at 77.47 146.05 0)
+			(at 69.85 146.05 0)
 			(effects
 				(font
@@
 		)
 		(property "Description" "Power symbol creates a global label with name \"GND\" , ground"
-			(at 77.47 146.05 0)
+			(at 69.85 146.05 0)
 			(effects
 				(font
@@
 					(unit 1)
 				)
+			)
+		)
+	)
+	(symbol
+		(lib_id "Device:D_TVS_Filled")
+		(at 77.47 142.24 90)
+		(unit 1)
+		(exclude_from_sim no)
+		(in_bom yes)
+		(on_board yes)
+		(dnp no)
+		(property "Reference" "D2"
+			(at 80.01 140.9699 90)
+			(effects
+				(font
+					(size 1.27 1.27)
+				)
+				(justify right)
+			)
+		)
+		(property "Value" "TVS"
+			(at 80.01 143.5099 90)
+			(effects
+				(font
+					(size 1.27 1.27)
+				)
+				(justify right)
+			)
+		)
+		(property "Footprint" "Diode_SMD:D_SMA"
+			(at 77.47 142.24 0)
+			(effects
+				(font
+					(size 1.27 1.27)
+				)
+				(hide yes)
+			)
+		)
+		(property "Datasheet" "~"
+			(at 77.47 142.24 0)
+			(effects
+				(font
+					(size 1.27 1.27)
+				)
+				(hide yes)
+			)
+		)
+		(property "Description" "Bidirectional transient-voltage-suppression diode, filled shape"
+			(at 77.47 142.24 0)
+			(effects
+				(font
+					(size 1.27 1.27)
+				)
+				(hide yes)
+			)
+		)
+		(pin "1"
+		)
+		(pin "2"
+		)
+		(instances
+			(project "lora"
+				(path "/e7e6f94f-519b-4ec5-b32e-6265e8eb4710"
+					(reference "D2")
+					(unit 1)
+				)

Commit message: update step
Parts:
- R4: value 1k -> 100
Changed lines of the file:
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@@
 			)
 		)
-		(property "Value" "1k"
+		(property "Value" "100"
 			(at 122.428 175.006 0)
 			(effects
